File: inrush-limiter/main.sch (KiCad schematic (older format))
At the start: 8 parts

Commit message: update
Parts:
- added C?: 100uF, 25V, symbol CP
- added C?: 3.3uF, symbol CP
- added D?: ZENER, symbol ZENER
- added K?: RELAY_2RT, symbol RELAY_2RT
- added P?: CONN_01X04, symbol CONN_01X04
- added Q? (x2): PN2222A, symbol PN2222A
- added R?: 2k, symbol R
- added R?: 100, symbol R
- added R?: 1000, symbol R
- added R?: 10K, symbol R
- added R?: 50K, symbol R
- added R?: 100K, symbol R
- added R?: 1M, symbol R
- added U?: LM393, symbol LM393
Connections:
- net labels added: +5V, GND, we-want-test-points
- wire segments 20 -> 49

Commit message: looks ok
Parts:
- removed P?: CONN_01X04, symbol CONN_01X04
- added R?: R, symbol R
- P?: value CONN_01X05 -> CONN_01X06; symbol CONN_01X05 -> CONN_01X06
Connections:
- net labels added: AC-live, AC-live-f, AC-live-out, AC-neut
- net labels removed: we-want-test-points
- wire segments 49 -> 61
Other:
- moved on the sheet: C?, D?, F?, K?, Q?, R?, U?A

Commit message: add isolation resistor
Parts:
- added R?: 0, symbol R
- C?: value 47nF -> 47nF, x2
Connections:
- wire segments 61 -> 62
Changed lines of the file:
@@
 P 2100 2250
 F 0 "C?" H 2125 2350 50  0000 L CNN
-F 1 "47nF" H 2125 2150 50  0000 L CNN
+F 1 "47nF, x2" H 2125 2150 50  0000 L CNN
 F 2 "" H 2138 2100 50  0000 C CNN
 F 3 "" H 2100 2250 50  0000 C CNN
@@
 L +5V #PWR?
 U 1 1 57C1B997
-P 1150 3950
-F 0 "#PWR?" H 1150 3800 50  0001 C CNN
-F 1 "+5V" H 1150 4090 50  0000 C CNN
-F 2 "" H 1150 3950 50  0000 C CNN
-F 3 "" H 1150 3950 50  0000 C CNN
-	1    1150 3950
+P 1150 3550
+F 0 "#PWR?" H 1150 3400 50  0001 C CNN
+F 1 "+5V" H 1150 3690 50  0000 C CNN
+F 2 "" H 1150 3550 50  0000 C CNN
+F 3 "" H 1150 3550 50  0000 C CNN
+	1    1150 3550
 	1    0    0    -1
 $EndComp
@@
 Connection ~ 2500 5350
 Wire Wire Line
-	1150 3950 1150 4200
+	1150 4000 1150 4200
 Connection ~ 1750 4100
 Wire Wire Line
@@
 	6200 4500 6000 4500
 Connection ~ 6200 4300
+$Comp
+L R R?
+U 1 1 57C35DF4
+P 1150 3850
+F 0 "R?" V 1230 3850 50  0000 C CNN
+F 1 "0" V 1150 3850 50  0000 C CNN
+F 2 "" V 1080 3850 50  0000 C CNN
+F 3 "" H 1150 3850 50  0000 C CNN
+	1    1150 3850
+	1    0    0    -1
+$EndComp
+Wire Wire Line
+	1150 3550 1150 3700
 $EndSCHEMATC

Commit message: tidy
Connections:
- wire segments 62 -> 63
Other:
- moved on the sheet: R?
Changed lines of the file:
@@
 L R R?
 U 1 1 57C14D32
-P 2000 3050
-F 0 "R?" V 2080 3050 50  0000 C CNN
-F 1 "100" V 2000 3050 50  0000 C CNN
-F 2 "" V 1930 3050 50  0000 C CNN
-F 3 "" H 2000 3050 50  0000 C CNN
-	1    2000 3050
+P 2100 3050
+F 0 "R?" V 2180 3050 50  0000 C CNN
+F 1 "100" V 2100 3050 50  0000 C CNN
+F 2 "" V 2030 3050 50  0000 C CNN
+F 3 "" H 2100 3050 50  0000 C CNN
+	1    2100 3050
 	0    1    1    0
 $EndComp
@@
 L GND #PWR?
 U 1 1 57C1A76B
-P 4950 3650
-F 0 "#PWR?" H 4950 3400 50  0001 C CNN
-F 1 "GND" H 4950 3500 50  0000 C CNN
-F 2 "" H 4950 3650 50  0000 C CNN
-F 3 "" H 4950 3650 50  0000 C CNN
-	1    4950 3650
+P 4950 3700
+F 0 "#PWR?" H 4950 3450 50  0001 C CNN
+F 1 "GND" H 4950 3550 50  0000 C CNN
+F 2 "" H 4950 3700 50  0000 C CNN
+F 3 "" H 4950 3700 50  0000 C CNN
+	1    4950 3700
 	1    0    0    -1
 $EndComp
@@
 	2650 2650 2550 2650
 Wire Wire Line
-	2550 2650 2550 3450
+	2550 2650 2550 3550
 Connection ~ 2650 2650
 Wire Wire Line
@@
 	4400 3050 4400 3150
 Wire Wire Line
-	2550 3450 4950 3450
+	2550 3550 4950 3550
 Wire Wire Line
 	4400 3100 4650 3100
@@
 Connection ~ 4400 2650
 Wire Wire Line
-	4950 3300 4950 3650
-Connection ~ 4400 3450
-Wire Wire Line
-	3750 3050 3750 3450
-Connection ~ 3750 3450
-Connection ~ 4950 3450
-Wire Wire Line
-	3000 3050 2150 3050
+	4950 3300 4950 3700
+Wire Wire Line
+	3750 3550 3750 3050
+Connection ~ 3750 3550
+Wire Wire Line
+	3000 3050 2250 3050
 Wire Wire Line
 	2900 4750 3000 4750
@@
 	3700 5350 3700 4950
 Wire Wire Line
-	1550 3050 1850 3050
+	1550 3050 1950 3050
 Wire Wire Line
 	4750 4400 4600 4400
@@
 Wire Wire Line
 	1150 3550 1150 3700
+Connection ~ 4950 3550
+Wire Wire Line
+	4400 3450 4400 3550
+Connection ~ 4400 3550
 $EndSCHEMATC

Commit message: tidy
Connections:
- wire segments 63 -> 88
Other:
- moved on the sheet: C?, R?
Changed lines of the file:
@@
 L C C?
 U 1 1 57C0BEB1
-P 2100 2250
-F 0 "C?" H 2125 2350 50  0000 L CNN
-F 1 "47nF, x2" H 2125 2150 50  0000 L CNN
-F 2 "" H 2138 2100 50  0000 C CNN
-F 3 "" H 2100 2250 50  0000 C CNN
-	1    2100 2250
+P 2050 2250
+F 0 "C?" H 2075 2350 50  0000 L CNN
+F 1 "47nF, x2" H 2075 2150 50  0000 L CNN
+F 2 "" H 2088 2100 50  0000 C CNN
+F 3 "" H 2050 2250 50  0000 C CNN
+	1    2050 2250
 	0    1    1    0
 $EndComp
@@
 L R R?
 U 1 1 57C0BED5
-P 2100 2700
-F 0 "R?" V 2180 2700 50  0000 C CNN
-F 1 "470k" V 2100 2700 50  0000 C CNN
-F 2 "" V 2030 2700 50  0000 C CNN
-F 3 "" H 2100 2700 50  0000 C CNN
-	1    2100 2700
+P 2050 2700
+F 0 "R?" V 2130 2700 50  0000 C CNN
+F 1 "470k" V 2050 2700 50  0000 C CNN
+F 2 "" V 1980 2700 50  0000 C CNN
+F 3 "" H 2050 2700 50  0000 C CNN
+	1    2050 2700
 	0    1    1    0
 $EndComp
@@
 L CP C?
 U 1 1 57C0C56F
-P 3750 2900
-F 0 "C?" H 3775 3000 50  0000 L CNN
-F 1 "100uF, 25V" H 3775 2800 50  0000 L CNN
-F 2 "" H 3788 2750 50  0000 C CNN
-F 3 "" H 3750 2900 50  0000 C CNN
-	1    3750 2900
+P 3750 3050
+F 0 "C?" H 3775 3150 50  0000 L CNN
+F 1 "100uF, 25V" H 3775 2950 50  0000 L CNN
+F 2 "" H 3788 2900 50  0000 C CNN
+F 3 "" H 3750 3050 50  0000 C CNN
+	1    3750 3050
 	1    0    0    -1
 $EndComp
@@
 L R R?
 U 1 1 57C14D32
-P 2100 3050
-F 0 "R?" V 2180 3050 50  0000 C CNN
-F 1 "100" V 2100 3050 50  0000 C CNN
-F 2 "" V 2030 3050 50  0000 C CNN
-F 3 "" H 2100 3050 50  0000 C CNN
-	1    2100 3050
+P 2050 3050
+F 0 "R?" V 2130 3050 50  0000 C CNN
+F 1 "100" V 2050 3050 50  0000 C CNN
+F 2 "" V 1980 3050 50  0000 C CNN
+F 3 "" H 2050 3050 50  0000 C CNN
+	1    2050 3050
 	0    1    1    0
 $EndComp
@@
 L GND #PWR?
 U 1 1 57C1A76B
-P 4950 3700
-F 0 "#PWR?" H 4950 3450 50  0001 C CNN
-F 1 "GND" H 4950 3550 50  0000 C CNN
-F 2 "" H 4950 3700 50  0000 C CNN
-F 3 "" H 4950 3700 50  0000 C CNN
-	1    4950 3700
+P 4950 3750
+F 0 "#PWR?" H 4950 3500 50  0001 C CNN
+F 1 "GND" H 4950 3600 50  0000 C CNN
+F 2 "" H 4950 3750 50  0000 C CNN
+F 3 "" H 4950 3750 50  0000 C CNN
+	1    4950 3750
 	1    0    0    -1
 $EndComp
@@
 $EndComp
 Wire Wire Line
-	1600 2250 1950 2250
-Wire Wire Line
-	1850 2250 1850 2700
-Wire Wire Line
-	1850 2700 1950 2700
-Connection ~ 1850 2250
-Wire Wire Line
-	2250 2250 3000 2250
-Wire Wire Line
-	2250 2700 2400 2700
-Wire Wire Line
-	2400 2700 2400 2250
-Connection ~ 2400 2250
+	1550 2250 1800 2250
+Wire Wire Line
+	1800 2250 1900 2250
+Wire Wire Line
+	1800 2250 1800 2700
+Wire Wire Line
+	1800 2700 1900 2700
+Connection ~ 1800 2250
+Wire Wire Line
+	2200 2250 2350 2250
+Wire Wire Line
+	2350 2250 2950 2250
+Wire Wire Line
+	2200 2700 2350 2700
+Wire Wire Line
+	2350 2700 2350 2250
+Connection ~ 2350 2250
 Wire Wire Line
 	3000 2250 3000 2450
 Wire Wire Line
-	2950 2450 3050 2450
+	2950 2450 3000 2450
+Wire Wire Line
+	3000 2450 3050 2450
 Connection ~ 3000 2450
 Wire Wire Line
-	2650 2450 2650 2850
-Wire Wire Line
-	3350 2450 3350 2850
-Wire Wire Line
-	2950 2850 3050 2850
+	2650 2450 2650 2650
+Wire Wire Line
+	2650 2650 2650 2850
+Wire Wire Line
+	3350 2450 3350 2650
+Wire Wire Line
+	3350 2650 3350 2850
+Wire Wire Line
+	2950 2850 3000 2850
+Wire Wire Line
+	3000 2850 3050 2850
 Wire Wire Line
 	3000 3050 3000 2850
 Connection ~ 3000 2850
 Wire Wire Line
-	2650 2650 2550 2650
-Wire Wire Line
-	2550 2650 2550 3550
+	2650 2650 2500 2650
+Wire Wire Line
+	2500 2650 2500 3550
 Connection ~ 2650 2650
 Wire Wire Line
-	3350 2650 4950 2650
+	3350 2650 3750 2650
+Wire Wire Line
+	3750 2650 4400 2650
+Wire Wire Line
+	4400 2650 4950 2650
 Connection ~ 3350 2650
 Wire Wire Line
-	3750 2650 3750 2750
+	3750 2650 3750 2900
 Connection ~ 3750 2650
 Wire Wire Line
-	4400 3050 4400 3150
-Wire Wire Line
-	2550 3550 4950 3550
+	4400 3050 4400 3100
+Wire Wire Line
+	4400 3100 4400 3150
+Wire Wire Line
+	2500 3550 3750 3550
+Wire Wire Line
+	3750 3550 4400 3550
+Wire Wire Line
+	4400 3550 4950 3550
 Wire Wire Line
 	4400 3100 4650 3100
@@
 Connection ~ 4400 2650
 Wire Wire Line
-	4950 3300 4950 3700
-Wire Wire Line
-	3750 3550 3750 3050
+	4950 3300 4950 3550
+Wire Wire Line
+	4950 3550 4950 3750
+Wire Wire Line
+	3750 3550 3750 3200
 Connection ~ 3750 3550
 Wire Wire Line
-	3000 3050 2250 3050
+	3000 3050 2200 3050
 Wire Wire Line
 	2900 4750 3000 4750
@@
 	3300 4750 3400 4750
 Wire Wire Line
-	1150 4100 4750 4100
-Wire Wire Line
-	1750 4500 1750 4950
+	1150 4100 1750 4100
+Wire Wire Line
+	1750 4100 2500 4100
+Wire Wire Line
+	2500 4100 4750 4100
+Wire Wire Line
+	1750 4500 1750 4850
+Wire Wire Line
+	1750 4850 1750 4950
 Wire Wire Line
 	2300 4850 1750 4850
@@
 	1750 5350 1750 5250
 Wire Wire Line
-	1150 5350 3700 5350
+	1150 5350 1450 5350
+Wire Wire Line
+	1450 5350 1750 5350
+Wire Wire Line
+	1750 5350 2500 5350
+Wire Wire Line
+	2500 5350 3700 5350
 Wire Wire Line
 	2500 5350 2500 5050
 Connection ~ 2500 5350
 Wire Wire Line
-	1150 4000 1150 4200
+	1150 4000 1150 4100
+Wire Wire Line
+	1150 4100 1150 4200
 Connection ~ 1750 4100
 Wire Wire Line
-	1150 4500 1150 4950
-Wire Wire Line
-	1150 5250 1150 5500
+	1150 4500 1150 4650
+Wire Wire Line
+	1150 4650 1150 4950
+Wire Wire Line
+	1150 5250 1150 5350
+Wire Wire Line
+	1150 5350 1150 5500
 Connection ~ 1750 5350
 Connection ~ 1150 5350
 Wire Wire Line
-	1150 4650 2300 4650
+	1150 4650 1450 4650
+Wire Wire Line
+	1450 4650 2300 4650
 Connection ~ 1150 4650
 Wire Wire Line
@@
 	3700 5350 3700 4950
 Wire Wire Line
-	1550 3050 1950 3050
+	1550 3050 1900 3050
 Wire Wire Line
 	4750 4400 4600 4400
 Wire Wire Line
-	5550 4300 6450 4300
+	5550 4300 6200 4300
+Wire Wire Line
+	6200 4300 6450 4300
 Wire Wire Line
 	5550 4500 5700 4500
 Wire Wire Line
-	4950 2450 4950 2900
+	4950 2450 4950 2650
+Wire Wire Line
+	4950 2650 4950 2900
 Connection ~ 4950 2650
 Text GLabel 6450 4300 2    60   Input ~ 0
@@
 AC-live-out
 Wire Wire Line
-	1350 1050 1950 1050
+	1350 1050 1700 1050
+Wire Wire Line
+	1700 1050 1950 1050
 Wire Wire Line
 	1650 1850 1500 1850
