File: inrush-limiter/main.sch (KiCad schematic (older format))
At the start: 24 parts

Commit message: start of pcb
Parts:
- C1: renamed from C?; footprint (none) -> Capacitors_ThroughHole:C_Radial_D5_L6_P2.5
- C2: renamed from C?; footprint (none) -> Capacitors_ThroughHole:C_Rect_L13_W4_P10
- C3: renamed from C?; footprint (none) -> Capacitors_ThroughHole:C_Radial_D10_L16_P5
- gave numbers to parts that had none: 21
Connections:
- wire segments 88 -> 63

Commit message: fix relay footprint and reimport
Parts:
- removed K1: RELAY_2RT, symbol RELAY_2RT
- added K?: RELAY_2RT, symbol RELAY_2RT
- C2: footprint Capacitors_ThroughHole:C_Rect_L13_W4_P10 -> Capacitors_ThroughHole:C_Rect_L18_W5_P15
- C3: footprint Capacitors_ThroughHole:C_Radial_D10_L16_P5 -> Capacitors_ThroughHole:C_Radial_D8_L13_P3.8
- D1, D2, D3, D4: footprint (none) -> Diodes_ThroughHole:Diode_DO-35_SOD27_Horizontal_RM10; symbol D -> 1N4007
- D5: footprint (none) -> Diodes_ThroughHole:Diode_DO-35_SOD27_Horizontal_RM10
- F1: footprint (none) -> Fuse_Holders_and_Fuses:Fuseholder5x20_horiz_SemiClosed_Casing10x25mm
- P1: footprint (none) -> Pin_Headers:Pin_Header_Straight_1x06
- Q1, Q2: footprint (none) -> TO_SOT_Packages_THT:TO-92_Inline_Narrow_Oval
- R1, R2, R3, R4, R5, R6, R7, R9: footprint (none) -> Resistors_ThroughHole:Resistor_Horizontal_RM7mm
- R10: value R -> 100, 5W; footprint (none) -> Resistors_ThroughHole:Resistor_Horizontal_RM25mm
- R8: value 1000 -> 1K; footprint (none) -> Resistors_ThroughHole:Resistor_Horizontal_RM7mm
- U1: footprint (none) -> Housings_DIP:DIP-8_W7.62mm_LongPads
Connections:
- wire segments 63 -> 88
Changed lines of the file:
@@
 EESchema Schematic File Version 2
+LIBS:my
+LIBS:Carlolib-disc
 LIBS:power
 LIBS:device
@@
 LIBS:contrib
 LIBS:valves
-LIBS:Carlolib-disc
 LIBS:main-cache
 EELAYER 25 0
@@
 F 0 "C2" H 2075 2350 50  0000 L CNN
 F 1 "47nF, x2" H 2075 2150 50  0000 L CNN
-F 2 "Capacitors_ThroughHole:C_Rect_L13_W4_P10" H 2088 2100 50  0001 C CNN
+F 2 "Capacitors_ThroughHole:C_Rect_L18_W5_P15" H 2088 2100 50  0001 C CNN
 F 3 "" H 2050 2250 50  0000 C CNN
 	1    2050 2250
@@
 F 0 "R6" V 2130 2700 50  0000 C CNN
 F 1 "470k" V 2050 2700 50  0000 C CNN
-F 2 "" V 1980 2700 50  0001 C CNN
+F 2 "Resistors_ThroughHole:Resistor_Horizontal_RM7mm" V 1980 2700 50  0001 C CNN
 F 3 "" H 2050 2700 50  0000 C CNN
 	1    2050 2700
@@
 F 0 "P1" H 1150 1500 50  0000 C CNN
 F 1 "CONN_01X06" V 1250 1200 50  0000 C CNN
-F 2 "" H 1150 1200 50  0001 C CNN
+F 2 "Pin_Headers:Pin_Header_Straight_1x06" H 1150 1200 50  0001 C CNN
 F 3 "" H 1150 1200 50  0000 C CNN
 	1    1150 1200
@@
 F 0 "F1" H 2000 1900 50  0000 C CNN
 F 1 "FUSE" H 1800 1800 50  0000 C CNN
-F 2 "" H 1900 1850 50  0001 C CNN
+F 2 "Fuse_Holders_and_Fuses:Fuseholder5x20_horiz_SemiClosed_Casing10x25mm" H 1900 1850 50  0001 C CNN
 F 3 "" H 1900 1850 50  0000 C CNN
 	1    1900 1850
@@
 $EndComp
 $Comp
-L D D1
+L 1N4007 D1
 U 1 1 57C0C128
 P 2800 2450
 F 0 "D1" H 2800 2550 50  0000 C CNN
 F 1 "D" H 2800 2350 50  0000 C CNN
-F 2 "" H 2800 2450 50  0001 C CNN
+F 2 "Diodes_ThroughHole:Diode_DO-35_SOD27_Horizontal_RM10" H 2800 2450 50  0001 C CNN
 F 3 "" H 2800 2450 50  0000 C CNN
 	1    2800 2450
-	-1   0    0    1
-$EndComp
-$Comp
-L D D3
+	1    0    0    -1
+$EndComp
+$Comp
+L 1N4007 D3
 U 1 1 57C0C217
 P 3200 2450
 F 0 "D3" H 3200 2550 50  0000 C CNN
 F 1 "D" H 3200 2350 50  0000 C CNN
-F 2 "" H 3200 2450 50  0001 C CNN
+F 2 "Diodes_ThroughHole:Diode_DO-35_SOD27_Horizontal_RM10" H 3200 2450 50  0001 C CNN
 F 3 "" H 3200 2450 50  0000 C CNN
 	1    3200 2450
-	-1   0    0    1
-$EndComp
-$Comp
-L D D2
+	1    0    0    -1
+$EndComp
+$Comp
+L 1N4007 D2
 U 1 1 57C0C23E
 P 2800 2850
 F 0 "D2" H 2800 2950 50  0000 C CNN
 F 1 "D" H 2800 2750 50  0000 C CNN
-F 2 "" H 2800 2850 50  0001 C CNN
+F 2 "Diodes_ThroughHole:Diode_DO-35_SOD27_Horizontal_RM10" H 2800 2850 50  0001 C CNN
 F 3 "" H 2800 2850 50  0000 C CNN
 	1    2800 2850
-	-1   0    0    1
-$EndComp
-$Comp
-L D D4
+	1    0    0    -1
+$EndComp
+$Comp
+L 1N4007 D4
 U 1 1 57C0C26B
 P 3200 2850
 F 0 "D4" H 3200 2950 50  0000 C CNN
 F 1 "D" H 3200 2750 50  0000 C CNN
-F 2 "" H 3200 2850 50  0001 C CNN
+F 2 "Diodes_ThroughHole:Diode_DO-35_SOD27_Horizontal_RM10" H 3200 2850 50  0001 C CNN
 F 3 "" H 3200 2850 50  0000 C CNN
 	1    3200 2850
-	-1   0    0    1
+	1    0    0    -1
 $EndComp
 $Comp
@@
 F 0 "C3" H 3775 3150 50  0000 L CNN
 F 1 "100uF, 25V" H 3775 2950 50  0000 L CNN
-F 2 "Capacitors_ThroughHole:C_Radial_D10_L16_P5" H 3788 2900 50  0001 C CNN
+F 2 "Capacitors_ThroughHole:C_Radial_D8_L13_P3.8" H 3788 2900 50  0001 C CNN
 F 3 "" H 3750 3050 50  0000 C CNN
 	1    3750 3050
@@
 F 0 "D5" H 4400 2950 50  0000 C CNN
 F 1 "ZENER" H 4400 2750 50  0000 C CNN
-F 2 "" H 4400 2850 50  0001 C CNN
+F 2 "Diodes_ThroughHole:Diode_DO-35_SOD27_Horizontal_RM10" H 4400 2850 50  0001 C CNN
 F 3 "" H 4400 2850 50  0000 C CNN
 	1    4400 2850
@@
 F 0 "R9" V 4480 3300 50  0000 C CNN
 F 1 "2k" V 4400 3300 50  0000 C CNN
-F 2 "" V 4330 3300 50  0001 C CNN
+F 2 "Resistors_ThroughHole:Resistor_Horizontal_RM7mm" V 4330 3300 50  0001 C CNN
 F 3 "" H 4400 3300 50  0000 C CNN
 	1    4400 3300
@@
 F 0 "Q2" H 5050 3175 50  0000 L CNN
 F 1 "PN2222A" H 5050 3100 50  0000 L CNN
-F 2 "" H 5050 3025 50  0001 L CIN
+F 2 "TO_SOT_Packages_THT:TO-92_Inline_Narrow_Oval" H 5050 3025 50  0001 L CIN
 F 3 "" H 4850 3100 50  0000 L CNN
 	1    4850 3100
@@
 F 0 "R7" V 2130 3050 50  0000 C CNN
 F 1 "100" V 2050 3050 50  0000 C CNN
-F 2 "" V 1980 3050 50  0001 C CNN
+F 2 "Resistors_ThroughHole:Resistor_Horizontal_RM7mm" V 1980 3050 50  0001 C CNN
 F 3 "" H 2050 3050 50  0000 C CNN
 	1    2050 3050
@@
 F 0 "U1" H 2750 4900 50  0000 C CNN
 F 1 "LM393" H 2850 4600 50  0000 C CNN
-F 2 "" H 2600 4750 50  0001 C CNN
+F 2 "Housings_DIP:DIP-8_W7.62mm_LongPads" H 2600 4750 50  0001 C CNN
 F 3 "" H 2600 4750 50  0000 C CNN
 	1    2600 4750
@@
 F 0 "Q1" H 3800 4825 50  0000 L CNN
 F 1 "PN2222A" H 3800 4750 50  0000 L CNN
-F 2 "" H 3800 4675 50  0001 L CIN
+F 2 "TO_SOT_Packages_THT:TO-92_Inline_Narrow_Oval" H 3800 4675 50  0001 L CIN
 F 3 "" H 3600 4750 50  0000 L CNN
 	1    3600 4750
@@
 P 3150 4750
 F 0 "R8" V 3230 4750 50  0000 C CNN
-F 1 "1000" V 3150 4750 50  0000 C CNN
-F 2 "" V 3080 4750 50  0001 C CNN
+F 1 "1K" V 3150 4750 50  0000 C CNN
+F 2 "Resistors_ThroughHole:Resistor_Horizontal_RM7mm" V 3080 4750 50  0001 C CNN
 F 3 "" H 3150 4750 50  0000 C CNN
 	1    3150 4750
 	0    1    1    0
-$EndComp
-$Comp
-L RELAY_2RT K1
-U 1 1 57C1BDD5
-P 5150 4450
-F 0 "K1" H 5100 4850 50  0000 C CNN
-F 1 "RELAY_2RT" H 5300 3950 50  0000 C CNN
-F 2 "" H 5150 4450 50  0001 C CNN
-F 3 "" H 5150 4450 50  0000 C CNN
-	1    5150 4450
-	1    0    0    1
 $EndComp
 $Comp
@@
 F 0 "R4" V 1830 4350 50  0000 C CNN
 F 1 "10K" V 1750 4350 50  0000 C CNN
-F 2 "" V 1680 4350 50  0001 C CNN
+F 2 "Resistors_ThroughHole:Resistor_Horizontal_RM7mm" V 1680 4350 50  0001 C CNN
 F 3 "" H 1750 4350 50  0000 C CNN
 	1    1750 4350
@@
 F 0 "R5" V 1830 5100 50  0000 C CNN
 F 1 "50K" V 1750 5100 50  0000 C CNN
-F 2 "" V 1680 5100 50  0001 C CNN
+F 2 "Resistors_ThroughHole:Resistor_Horizontal_RM7mm" V 1680 5100 50  0001 C CNN
 F 3 "" H 1750 5100 50  0000 C CNN
 	1    1750 5100
@@
 F 0 "R2" V 1230 4350 50  0000 C CNN
 F 1 "100K" V 1150 4350 50  0000 C CNN
-F 2 "" V 1080 4350 50  0001 C CNN
+F 2 "Resistors_ThroughHole:Resistor_Horizontal_RM7mm" V 1080 4350 50  0001 C CNN
 F 3 "" H 1150 4350 50  0000 C CNN
 	1    1150 4350
@@
 F 0 "R3" V 1230 5100 50  0000 C CNN
 F 1 "1M" V 1150 5100 50  0000 C CNN
-F 2 "" V 1080 5100 50  0001 C CNN
+F 2 "Resistors_ThroughHole:Resistor_Horizontal_RM7mm" V 1080 5100 50  0001 C CNN
 F 3 "" H 1150 5100 50  0000 C CNN
 	1    1150 5100
@@
 P 5850 4500
 F 0 "R10" V 5930 4500 50  0000 C CNN
-F 1 "R" V 5850 4500 50  0000 C CNN
-F 2 "" V 5780 4500 50  0001 C CNN
+F 1 "100, 5W" V 5850 4500 50  0000 C CNN
+F 2 "Resistors_ThroughHole:Resistor_Horizontal_RM25mm" V 5780 4500 50  0001 C CNN
 F 3 "" H 5850 4500 50  0000 C CNN
 	1    5850 4500
@@
 $EndComp
 Wire Wire Line
-	1550 2250 1900 2250
+	1550 2250 1800 2250
+Wire Wire Line
+	1800 2250 1900 2250
 Wire Wire Line
 	1800 2250 1800 2700
@@
 Connection ~ 1800 2250
 Wire Wire Line
-	2200 2250 3000 2250
+	2200 2250 2350 2250
+Wire Wire Line
+	2350 2250 3000 2250
 Wire Wire Line
 	2200 2700 2350 2700
@@
 	3000 2250 3000 2450
 Wire Wire Line
-	2950 2450 3050 2450
+	2950 2450 3000 2450
+Wire Wire Line
+	3000 2450 3050 2450
 Connection ~ 3000 2450
 Wire Wire Line
-	2650 2450 2650 2850
-Wire Wire Line
-	3350 2450 3350 2850
-Wire Wire Line
-	2950 2850 3050 2850
+	2650 2450 2650 2650
+Wire Wire Line
+	2650 2650 2650 2850
+Wire Wire Line
+	3350 2450 3350 2650
+Wire Wire Line
+	3350 2650 3350 2850
+Wire Wire Line
+	2950 2850 3000 2850
+Wire Wire Line
+	3000 2850 3050 2850
 Wire Wire Line
 	3000 3050 3000 2850
@@
 Connection ~ 2650 2650
 Wire Wire Line
-	3350 2650 4950 2650
+	3350 2650 3750 2650
+Wire Wire Line
+	3750 2650 4400 2650
+Wire Wire Line
+	4400 2650 4950 2650
 Connection ~ 3350 2650
 Wire Wire Line
@@
 Connection ~ 3750 2650
 Wire Wire Line
-	4400 3050 4400 3150
-Wire Wire Line
-	2500 3550 4950 3550
+	4400 3050 4400 3100
+Wire Wire Line
+	4400 3100 4400 3150
+Wire Wire Line
+	2500 3550 3750 3550
+Wire Wire Line
+	3750 3550 4400 3550
+Wire Wire Line
+	4400 3550 4950 3550
 Wire Wire Line
 	4400 3100 4650 3100
@@
 Connection ~ 4400 2650
 Wire Wire Line
-	4950 3300 4950 3750
+	4950 3300 4950 3550
+Wire Wire Line
+	4950 3550 4950 3750
 Wire Wire Line
 	3750 3550 3750 3200
@@
 	3300 4750 3400 4750
 Wire Wire Line
-	1150 4100 4750 4100
-Wire Wire Line
-	1750 4500 1750 4950
+	1150 4100 1750 4100
+Wire Wire Line
+	1750 4100 2500 4100
+Wire Wire Line
+	2500 4100 4750 4100
+Wire Wire Line
+	1750 4500 1750 4850
+Wire Wire Line
+	1750 4850 1750 4950
 Wire Wire Line
 	2300 4850 1750 4850
@@
 	1750 5350 1750 5250
 Wire Wire Line
-	1150 5350 3700 5350
+	1150 5350 1450 5350
+Wire Wire Line
+	1450 5350 1750 5350
+Wire Wire Line
+	1750 5350 2500 5350
+Wire Wire Line
+	2500 5350 3700 5350
 Connection ~ 2500 5350
 Wire Wire Line
-	1150 4000 1150 4200
+	1150 4000 1150 4100
+Wire Wire Line
+	1150 4100 1150 4200
 Connection ~ 1750 4100
 Wire Wire Line
-	1150 4500 1150 4950
-Wire Wire Line
-	1150 5250 1150 5500
+	1150 4500 1150 4650
+Wire Wire Line
+	1150 4650 1150 4950
+Wire Wire Line
+	1150 5250 1150 5350
+Wire Wire Line
+	1150 5350 1150 5500
 Connection ~ 1750 5350
 Connection ~ 1150 5350
 Wire Wire Line
-	1150 4650 2300 4650
+	1150 4650 1450 4650
+Wire Wire Line
+	1450 4650 2300 4650
 Connection ~ 1150 4650
 Connection ~ 2500 4100
@@
 	4750 4400 4600 4400
 Wire Wire Line
-	5550 4300 6450 4300
+	5550 4300 6200 4300
+Wire Wire Line
+	6200 4300 6450 4300
 Wire Wire Line
 	5550 4500 5700 4500
 Wire Wire Line
-	4950 2450 4950 2900
+	4950 2450 4950 2650
+Wire Wire Line
+	4950 2650 4950 2900
 Connection ~ 4950 2650
 Text GLabel 6450 4300 2    60   Input ~ 0
@@
 AC-live-out
 Wire Wire Line
-	1350 1050 1950 1050
+	1350 1050 1700 1050
+Wire Wire Line
+	1700 1050 1950 1050
 Wire Wire Line
 	1650 1850 1500 1850
@@
 F 0 "R1" V 1230 3850 50  0000 C CNN
 F 1 "0" V 1150 3850 50  0000 C CNN
-F 2 "" V 1080 3850 50  0001 C CNN
+F 2 "Resistors_ThroughHole:Resistor_Horizontal_RM7mm" V 1080 3850 50  0001 C CNN
 F 3 "" H 1150 3850 50  0000 C CNN
 	1    1150 3850
@@
 Wire Wire Line
 	2500 4450 2500 4100
+$Comp
+L RELAY_2RT K?
+U 1 1 57C3B514
+P 5150 4450
+F 0 "K?" H 5100 4850 50  0000 C CNN
+F 1 "RELAY_2RT" H 5300 3950 50  0000 C CNN
+F 2 "" H 5150 4450 50  0000 C CNN
+F 3 "" H 5150 4450 50  0000 C CNN
+	1    5150 4450
+	1    0    0    1
+$EndComp
 $EndSCHEMATC

Commit message: update
Parts:
- removed P1: CONN_01X06, Pin_Headers:Pin_Header_Straight_1x06, symbol CONN_01X06
- added P2: CONN_01X02, Pin_Headers:Pin_Header_Straight_1x02, symbol CONN_01X02
- added P?: CONN_01X04, symbol CONN_01X04
- K1: renamed from K?; footprint (none) -> Relays_ThroughHole:Relay_DPDT_Schrack-RT2_RM5mm
Connections:
- wire segments 88 -> 86
Changed lines of the file:
@@
-$EndComp
-$Comp
-L CONN_01X06 P1
-U 1 1 57C0BF7B
-P 1150 1200
-F 0 "P1" H 1150 1500 50  0000 C CNN
-F 1 "CONN_01X06" V 1250 1200 50  0000 C CNN
-F 2 "Pin_Headers:Pin_Header_Straight_1x06" H 1150 1200 50  0001 C CNN
-F 3 "" H 1150 1200 50  0000 C CNN
-	1    1150 1200
-	-1   0    0    1
 $EndComp
 $Comp
@@
 Text GLabel 2300 1850 2    60   Input ~ 0
 AC-live-f
-Text GLabel 1550 2250 0    60   Input ~ 0
+Text GLabel 1600 2250 0    60   Input ~ 0
 AC-live-f
 Text GLabel 4600 4400 0    60   Input ~ 0
@@
 $EndComp
 Wire Wire Line
-	1550 2250 1800 2250
+	1600 2250 1800 2250
 Wire Wire Line
 	1800 2250 1900 2250
@@
 Text GLabel 6450 4300 2    60   Input ~ 0
 AC-live-out
-Text GLabel 1950 1050 2    60   Input ~ 0
+Text GLabel 2500 1450 2    60   Input ~ 0
 AC-neut
 Wire Wire Line
 	2300 1850 2150 1850
-Text GLabel 1950 1250 2    60   Input ~ 0
-AC-live-out
-Wire Wire Line
-	1350 1050 1700 1050
-Wire Wire Line
-	1700 1050 1950 1050
 Wire Wire Line
 	1650 1850 1500 1850
-Wire Wire Line
-	1700 1050 1700 1150
-Wire Wire Line
-	1700 1150 1350 1150
-Connection ~ 1700 1050
-Wire Wire Line
-	1950 1250 1350 1250
-Text GLabel 1950 850  2    60   Input ~ 0
+Text GLabel 1950 1150 2    60   Input ~ 0
 AC-live
 Wire Wire Line
-	1950 850  1700 850
-Wire Wire Line
-	1700 850  1700 950
-Wire Wire Line
-	1700 950  1350 950
+	1950 1150 1700 1150
+Wire Wire Line
+	1700 1150 1700 1250
+Wire Wire Line
+	1700 1250 1350 1250
 $Comp
 L +5V #PWR05
 U 1 1 57C33EC3
-P 2900 1250
-F 0 "#PWR05" H 2900 1100 50  0001 C CNN
-F 1 "+5V" H 2900 1390 50  0000 C CNN
-F 2 "" H 2900 1250 50  0000 C CNN
-F 3 "" H 2900 1250 50  0000 C CNN
-	1    2900 1250
+P 4250 1200
+F 0 "#PWR05" H 4250 1050 50  0001 C CNN
+F 1 "+5V" H 4250 1340 50  0000 C CNN
+F 2 "" H 4250 1200 50  0000 C CNN
+F 3 "" H 4250 1200 50  0000 C CNN
+	1    4250 1200
 	1    0    0    -1
 $EndComp
@@
 L GND #PWR06
 U 1 1 57C33F05
-P 2900 1550
-F 0 "#PWR06" H 2900 1300 50  0001 C CNN
-F 1 "GND" H 2900 1400 50  0000 C CNN
-F 2 "" H 2900 1550 50  0000 C CNN
-F 3 "" H 2900 1550 50  0000 C CNN
-	1    2900 1550
-	1    0    0    -1
-$EndComp
-Wire Wire Line
-	2900 1550 2900 1450
-Wire Wire Line
-	2900 1450 1350 1450
-Wire Wire Line
-	1350 1350 2900 1350
-Wire Wire Line
-	2900 1350 2900 1250
+P 4250 1500
+F 0 "#PWR06" H 4250 1250 50  0001 C CNN
+F 1 "GND" H 4250 1350 50  0000 C CNN
+F 2 "" H 4250 1500 50  0000 C CNN
+F 3 "" H 4250 1500 50  0000 C CNN
+	1    4250 1500
+	1    0    0    -1
+$EndComp
+Wire Wire Line
+	4250 1500 4250 1400
+Wire Wire Line
+	4250 1300 4250 1200
 Wire Wire Line
 	6200 4300 6200 4500
@@
 	2500 4450 2500 4100
 $Comp
-L RELAY_2RT K?
+L RELAY_2RT K1
 U 1 1 57C3B514
 P 5150 4450
-F 0 "K?" H 5100 4850 50  0000 C CNN
+F 0 "K1" H 5100 4850 50  0000 C CNN
 F 1 "RELAY_2RT" H 5300 3950 50  0000 C CNN
-F 2 "" H 5150 4450 50  0000 C CNN
+F 2 "Relays_ThroughHole:Relay_DPDT_Schrack-RT2_RM5mm" H 5150 4450 50  0001 C CNN
 F 3 "" H 5150 4450 50  0000 C CNN
 	1    5150 4450
 	1    0    0    1
 $EndComp
+Wire Wire Line
+	1350 1550 1550 1550
+Text GLabel 1550 1550 2    60   Input ~ 0
+AC-live-out
+Text GLabel 2100 1300 2    60   Input ~ 0
+AC-neut
+Wire Wire Line
+	1350 1450 1450 1450
+Wire Wire Line
+	1450 1450 1450 1350
+Wire Wire Line
+	1450 1350 2100 1300
+Wire Wire Line
+	2500 1450 1350 1350
+$Comp
+L CONN_01X02 P2
+U 1 1 57C3DE82
+P 4050 1350
+F 0 "P2" H 4050 1650 50  0000 C CNN
+F 1 "CONN_01X02" V 4150 1350 50  0000 C CNN
+F 2 "Pin_Headers:Pin_Header_Straight_1x02" H 4050 1350 50  0001 C CNN
+F 3 "" H 4050 1350 50  0000 C CNN
+	1    4050 1350
+	-1   0    0    1
+$EndComp
+$Comp
+L CONN_01X04 P?
+U 1 1 57C3EB1A
+P 1150 1400
+F 0 "P?" H 1150 1650 50  0000 C CNN
+F 1 "CONN_01X04" V 1250 1400 50  0000 C CNN
+F 2 "" H 1150 1400 50  0000 C CNN
+F 3 "" H 1150 1400 50  0000 C CNN
+	1    1150 1400
+	-1   0    0    1
+$EndComp
 $EndSCHEMATC
