File: inrush-limiter/main.sch (KiCad schematic (older format))
At the start: 25 parts, among them K1 RELAY_2RT, P2 CONN_01X02, Q1 PN2222A, Q2 PN2222A, U1 LM393

Commit message: update
Parts:
- P1: renamed from P?; footprint (none) -> Connect:AK300-4
Connections:
- net labels added: AC-live-f-low, AC-neut-low
- wire segments 86 -> 65
Changed lines of the file:
@@
 AC-live
 Text GLabel 1550 3050 0    60   Input ~ 0
-AC-neut
+AC-neut-low
 Text GLabel 2300 1850 2    60   Input ~ 0
 AC-live-f
 Text GLabel 1600 2250 0    60   Input ~ 0
-AC-live-f
+AC-live-f-low
 Text GLabel 4600 4400 0    60   Input ~ 0
 AC-live-f
@@
 	0    -1   -1   0
 $EndComp
-Wire Wire Line
-	1600 2250 1800 2250
-Wire Wire Line
-	1800 2250 1900 2250
-Wire Wire Line
-	1800 2250 1800 2700
-Wire Wire Line
-	1800 2700 1900 2700
-Connection ~ 1800 2250
-Wire Wire Line
-	2200 2250 2350 2250
-Wire Wire Line
-	2350 2250 3000 2250
-Wire Wire Line
-	2200 2700 2350 2700
-Wire Wire Line
-	2350 2700 2350 2250
-Connection ~ 2350 2250
-Wire Wire Line
-	3000 2250 3000 2450
-Wire Wire Line
-	2950 2450 3000 2450
-Wire Wire Line
-	3000 2450 3050 2450
-Connection ~ 3000 2450
-Wire Wire Line
-	2650 2450 2650 2650
-Wire Wire Line
-	2650 2650 2650 2850
-Wire Wire Line
-	3350 2450 3350 2650
-Wire Wire Line
-	3350 2650 3350 2850
-Wire Wire Line
-	2950 2850 3000 2850
-Wire Wire Line
-	3000 2850 3050 2850
-Wire Wire Line
-	3000 3050 3000 2850
-Connection ~ 3000 2850
-Wire Wire Line
-	2650 2650 2500 2650
-Wire Wire Line
-	2500 2650 2500 3550
-Connection ~ 2650 2650
-Wire Wire Line
-	3350 2650 3750 2650
-Wire Wire Line
-	3750 2650 4400 2650
-Wire Wire Line
-	4400 2650 4950 2650
-Connection ~ 3350 2650
-Wire Wire Line
-	3750 2650 3750 2900
-Connection ~ 3750 2650
-Wire Wire Line
-	4400 3050 4400 3100
-Wire Wire Line
-	4400 3100 4400 3150
-Wire Wire Line
-	2500 3550 3750 3550
-Wire Wire Line
-	3750 3550 4400 3550
-Wire Wire Line
-	4400 3550 4950 3550
-Wire Wire Line
-	4400 3100 4650 3100
-Connection ~ 4400 3100
-Connection ~ 4400 2650
-Wire Wire Line
-	4950 3300 4950 3550
-Wire Wire Line
-	4950 3550 4950 3750
-Wire Wire Line
-	3750 3550 3750 3200
-Connection ~ 3750 3550
-Wire Wire Line
-	3000 3050 2200 3050
-Wire Wire Line
-	2900 4750 3000 4750
-Wire Wire Line
-	3300 4750 3400 4750
-Wire Wire Line
-	1150 4100 1750 4100
-Wire Wire Line
-	1750 4100 2500 4100
-Wire Wire Line
-	2500 4100 4750 4100
-Wire Wire Line
-	1750 4500 1750 4850
-Wire Wire Line
-	1750 4850 1750 4950
-Wire Wire Line
-	2300 4850 1750 4850
-Connection ~ 1750 4850
-Wire Wire Line
-	1750 4100 1750 4200
-Wire Wire Line
-	1750 5350 1750 5250
-Wire Wire Line
-	1150 5350 1450 5350
-Wire Wire Line
-	1450 5350 1750 5350
-Wire Wire Line
-	1750 5350 2500 5350
-Wire Wire Line
-	2500 5350 3700 5350
-Connection ~ 2500 5350
-Wire Wire Line
-	1150 4000 1150 4100
-Wire Wire Line
-	1150 4100 1150 4200
-Connection ~ 1750 4100
-Wire Wire Line
-	1150 4500 1150 4650
-Wire Wire Line
-	1150 4650 1150 4950
-Wire Wire Line
-	1150 5250 1150 5350
-Wire Wire Line
-	1150 5350 1150 5500
-Connection ~ 1750 5350
-Connection ~ 1150 5350
-Wire Wire Line
-	1150 4650 1450 4650
-Wire Wire Line
-	1450 4650 2300 4650
-Connection ~ 1150 4650
-Connection ~ 2500 4100
-Wire Wire Line
-	1450 5250 1450 5350
-Connection ~ 1450 5350
-Wire Wire Line
-	1450 4950 1450 4650
-Connection ~ 1450 4650
-Connection ~ 1150 4100
-Wire Wire Line
-	4750 4200 3700 4200
-Wire Wire Line
-	3700 4200 3700 4550
-Wire Wire Line
-	3700 5350 3700 4950
-Wire Wire Line
-	1550 3050 1900 3050
-Wire Wire Line
-	4750 4400 4600 4400
-Wire Wire Line
-	5550 4300 6200 4300
-Wire Wire Line
-	6200 4300 6450 4300
-Wire Wire Line
-	5550 4500 5700 4500
-Wire Wire Line
-	4950 2450 4950 2650
-Wire Wire Line
-	4950 2650 4950 2900
-Connection ~ 4950 2650
 Text GLabel 6450 4300 2    60   Input ~ 0
 AC-live-out
 Text GLabel 2500 1450 2    60   Input ~ 0
-AC-neut
-Wire Wire Line
-	2300 1850 2150 1850
-Wire Wire Line
-	1650 1850 1500 1850
+AC-neut-low
 Text GLabel 1950 1150 2    60   Input ~ 0
 AC-live
-Wire Wire Line
-	1950 1150 1700 1150
-Wire Wire Line
-	1700 1150 1700 1250
-Wire Wire Line
-	1700 1250 1350 1250
 $Comp
 L +5V #PWR05
@@
 	1    0    0    -1
 $EndComp
-Wire Wire Line
-	4250 1500 4250 1400
-Wire Wire Line
-	4250 1300 4250 1200
-Wire Wire Line
-	6200 4300 6200 4500
-Wire Wire Line
-	6200 4500 6000 4500
-Connection ~ 6200 4300
 $Comp
 L R R1
@@
 	1    0    0    -1
 $EndComp
-Wire Wire Line
-	1150 3550 1150 3700
-Connection ~ 4950 3550
-Wire Wire Line
-	4400 3450 4400 3550
-Connection ~ 4400 3550
-Wire Wire Line
-	2500 5050 2500 5350
-Wire Wire Line
-	2500 4450 2500 4100
 $Comp
 L RELAY_2RT K1
@@
 	1    0    0    1
 $EndComp
-Wire Wire Line
-	1350 1550 1550 1550
 Text GLabel 1550 1550 2    60   Input ~ 0
 AC-live-out
-Text GLabel 2100 1300 2    60   Input ~ 0
+Text GLabel 2500 1250 2    60   Input ~ 0
 AC-neut
-Wire Wire Line
-	1350 1450 1450 1450
-Wire Wire Line
-	1450 1450 1450 1350
-Wire Wire Line
-	1450 1350 2100 1300
-Wire Wire Line
-	2500 1450 1350 1350
 $Comp
 L CONN_01X02 P2
@@
 $EndComp
 $Comp
-L CONN_01X04 P?
+L CONN_01X04 P1
 U 1 1 57C3EB1A
 P 1150 1400
-F 0 "P?" H 1150 1650 50  0000 C CNN
+F 0 "P1" H 1150 1650 50  0000 C CNN
 F 1 "CONN_01X04" V 1250 1400 50  0000 C CNN
-F 2 "" H 1150 1400 50  0000 C CNN
+F 2 "Connect:AK300-4" H 1150 1400 50  0001 C CNN
 F 3 "" H 1150 1400 50  0000 C CNN
 	1    1150 1400
 	-1   0    0    1
 $EndComp
+Text GLabel 2300 2050 2    60   Input ~ 0
+AC-live-f-low
+Wire Wire Line
+	1600 2250 1900 2250
+Wire Wire Line
+	1800 2250 1800 2700
+Wire Wire Line
+	1800 2700 1900 2700
+Connection ~ 1800 2250
+Wire Wire Line
+	2200 2250 3000 2250
+Wire Wire Line
+	2200 2700 2350 2700
+Wire Wire Line
+	2350 2700 2350 2250
+Connection ~ 2350 2250
+Wire Wire Line
+	3000 2250 3000 2450
+Wire Wire Line
+	2950 2450 3050 2450
+Connection ~ 3000 2450
+Wire Wire Line
+	2650 2450 2650 2850
+Wire Wire Line
+	3350 2450 3350 2850
+Wire Wire Line
+	2950 2850 3050 2850
+Wire Wire Line
+	3000 3050 3000 2850
+Connection ~ 3000 2850
+Wire Wire Line
+	2650 2650 2500 2650
+Wire Wire Line
+	2500 2650 2500 3550
+Connection ~ 2650 2650
+Wire Wire Line
+	3350 2650 4950 2650
+Connection ~ 3350 2650
+Wire Wire Line
+	3750 2650 3750 2900
+Connection ~ 3750 2650
+Wire Wire Line
+	4400 3050 4400 3150
+Wire Wire Line
+	2500 3550 4950 3550
+Wire Wire Line
+	4400 3100 4650 3100
+Connection ~ 4400 3100
+Connection ~ 4400 2650
+Wire Wire Line
+	4950 3300 4950 3750
+Wire Wire Line
+	3750 3550 3750 3200
+Connection ~ 3750 3550
+Wire Wire Line
+	3000 3050 2200 3050
+Wire Wire Line
+	2900 4750 3000 4750
+Wire Wire Line
+	3300 4750 3400 4750
+Wire Wire Line
+	1150 4100 4750 4100
+Wire Wire Line
+	1750 4500 1750 4950
+Wire Wire Line
+	2300 4850 1750 4850
+Connection ~ 1750 4850
+Wire Wire Line
+	1750 4100 1750 4200
+Wire Wire Line
+	1750 5350 1750 5250
+Wire Wire Line
+	1150 5350 3700 5350
+Connection ~ 2500 5350
+Wire Wire Line
+	1150 4000 1150 4200
+Connection ~ 1750 4100
+Wire Wire Line
+	1150 4500 1150 4950
+Wire Wire Line
+	1150 5250 1150 5500
+Connection ~ 1750 5350
+Connection ~ 1150 5350
+Wire Wire Line
+	1150 4650 2300 4650
+Connection ~ 1150 4650
+Connection ~ 2500 4100
+Wire Wire Line
+	1450 5250 1450 5350
+Connection ~ 1450 5350
+Wire Wire Line
+	1450 4950 1450 4650
+Connection ~ 1450 4650
+Connection ~ 1150 4100
+Wire Wire Line
+	4750 4200 3700 4200
+Wire Wire Line
+	3700 4200 3700 4550
+Wire Wire Line
+	3700 5350 3700 4950
+Wire Wire Line
+	1550 3050 1900 3050
+Wire Wire Line
+	4750 4400 4600 4400
+Wire Wire Line
+	5550 4300 6450 4300
+Wire Wire Line
+	5550 4500 5700 4500
+Wire Wire Line
+	4950 2450 4950 2900
+Connection ~ 4950 2650
+Wire Wire Line
+	2150 1850 2300 1850
+Wire Wire Line
+	1650 1850 1500 1850
+Wire Wire Line
+	1950 1150 1700 1150
+Wire Wire Line
+	1700 1150 1700 1250
+Wire Wire Line
+	1700 1250 1350 1250
+Wire Wire Line
+	4250 1500 4250 1400
+Wire Wire Line
+	4250 1300 4250 1200
+Wire Wire Line
+	6200 4300 6200 4500
+Wire Wire Line
+	6200 4500 6000 4500
+Connection ~ 6200 4300
+Wire Wire Line
+	1150 3550 1150 3700
+Connection ~ 4950 3550
+Wire Wire Line
+	4400 3450 4400 3550
+Connection ~ 4400 3550
+Wire Wire Line
+	2500 5050 2500 5350
+Wire Wire Line
+	2500 4450 2500 4100
+Wire Wire Line
+	1350 1550 1550 1550
+Wire Wire Line
+	2300 2050 2200 2050
+Wire Wire Line
+	2200 2050 2200 1850
+Connection ~ 2200 1850
+Wire Wire Line
+	2500 1250 1800 1250
+Wire Wire Line
+	1800 1250 1800 1350
+Wire Wire Line
+	1800 1350 1350 1350
+Wire Wire Line
+	2500 1450 1350 1450
+Wire Wire Line
+	1800 1300 1800 1450
+Connection ~ 1800 1450
+Connection ~ 1800 1300
 $EndSCHEMATC

Commit message: got track width separated by netlist using 0 resistor
Parts:
- added R?: R, symbol R
Connections:
- wire segments 65 -> 70
Changed lines of the file:
@@
 Text GLabel 2300 1850 2    60   Input ~ 0
 AC-live-f
-Text GLabel 1600 2250 0    60   Input ~ 0
-AC-live-f-low
 Text GLabel 4600 4400 0    60   Input ~ 0
 AC-live-f
@@
 Text GLabel 6450 4300 2    60   Input ~ 0
 AC-live-out
-Text GLabel 2500 1450 2    60   Input ~ 0
-AC-neut-low
 Text GLabel 1950 1150 2    60   Input ~ 0
 AC-live
@@
 Text GLabel 2300 2050 2    60   Input ~ 0
 AC-live-f-low
-Wire Wire Line
-	1600 2250 1900 2250
+$Comp
+L R R?
+U 1 1 57C402C2
+P 2250 1400
+F 0 "R?" V 2330 1400 50  0000 C CNN
+F 1 "R" V 2250 1400 50  0000 C CNN
+F 2 "" V 2180 1400 50  0000 C CNN
+F 3 "" H 2250 1400 50  0000 C CNN
+	1    2250 1400
+	0    1    1    0
+$EndComp
+Wire Wire Line
+	950  2250 1900 2250
 Wire Wire Line
 	1800 2250 1800 2700
@@
 	1800 1350 1350 1350
 Wire Wire Line
-	2500 1450 1350 1450
+	1800 1450 1350 1450
 Wire Wire Line
 	1800 1300 1800 1450
 Connection ~ 1800 1450
 Connection ~ 1800 1300
+Wire Wire Line
+	2500 1650 950  1650
+Wire Wire Line
+	950  1650 950  2250
+Wire Wire Line
+	2400 1400 2500 1400
+Wire Wire Line
+	2500 1400 2500 1650
+Wire Wire Line
+	2100 1400 1800 1400
+Connection ~ 1800 1400
 $EndSCHEMATC

Commit message: add gnd plane
Parts:
- added R12: 0, Resistors_ThroughHole:Resistor_Horizontal_RM7mm, symbol R
- R11: renamed from R?; value R -> 0; footprint (none) -> Resistors_ThroughHole:Resistor_Horizontal_RM7mm
Connections:
- net labels removed: AC-live
- wire segments 70 -> 64
Other:
- moved on the sheet: F1, R11
Changed lines of the file:
@@
 L FUSE F1
 U 1 1 57C0C016
-P 1900 1850
-F 0 "F1" H 2000 1900 50  0000 C CNN
-F 1 "FUSE" H 1800 1800 50  0000 C CNN
-F 2 "Fuse_Holders_and_Fuses:Fuseholder5x20_horiz_SemiClosed_Casing10x25mm" H 1900 1850 50  0001 C CNN
-F 3 "" H 1900 1850 50  0000 C CNN
-	1    1900 1850
+P 1650 900
+F 0 "F1" H 1750 950 50  0000 C CNN
+F 1 "FUSE" H 1550 850 50  0000 C CNN
+F 2 "Fuse_Holders_and_Fuses:Fuseholder5x20_horiz_SemiClosed_Casing10x25mm" H 1650 900 50  0001 C CNN
+F 3 "" H 1650 900 50  0000 C CNN
+	1    1650 900
 	-1   0    0    -1
 $EndComp
@@
 $EndComp
 $Comp
-L GND #PWR01
+L GND #PWR6
 U 1 1 57C1A76B
 P 4950 3750
-F 0 "#PWR01" H 4950 3500 50  0001 C CNN
+F 0 "#PWR6" H 4950 3500 50  0001 C CNN
 F 1 "GND" H 4950 3600 50  0000 C CNN
 F 2 "" H 4950 3750 50  0000 C CNN
@@
 $EndComp
 $Comp
-L +5V #PWR02
+L +5V #PWR5
 U 1 1 57C1A7D8
 P 4950 2450
-F 0 "#PWR02" H 4950 2300 50  0001 C CNN
+F 0 "#PWR5" H 4950 2300 50  0001 C CNN
 F 1 "+5V" H 4950 2590 50  0000 C CNN
 F 2 "" H 4950 2450 50  0000 C CNN
@@
 $EndComp
 $Comp
-L +5V #PWR03
+L +5V #PWR1
 U 1 1 57C1B997
 P 1150 3550
-F 0 "#PWR03" H 1150 3400 50  0001 C CNN
+F 0 "#PWR1" H 1150 3400 50  0001 C CNN
 F 1 "+5V" H 1150 3690 50  0000 C CNN
 F 2 "" H 1150 3550 50  0000 C CNN
@@
 $EndComp
 $Comp
-L GND #PWR04
+L GND #PWR2
 U 1 1 57C1BA06
 P 1150 5500
-F 0 "#PWR04" H 1150 5250 50  0001 C CNN
+F 0 "#PWR2" H 1150 5250 50  0001 C CNN
 F 1 "GND" H 1150 5350 50  0000 C CNN
 F 2 "" H 1150 5500 50  0000 C CNN
@@
 	1    0    0    -1
 $EndComp
-Text GLabel 1500 1850 0    60   Input ~ 0
-AC-live
 Text GLabel 1550 3050 0    60   Input ~ 0
 AC-neut-low
-Text GLabel 2300 1850 2    60   Input ~ 0
+Text GLabel 2500 900  2    60   Input ~ 0
 AC-live-f
 Text GLabel 4600 4400 0    60   Input ~ 0
@@
 Text GLabel 6450 4300 2    60   Input ~ 0
 AC-live-out
-Text GLabel 1950 1150 2    60   Input ~ 0
-AC-live
-$Comp
-L +5V #PWR05
+$Comp
+L +5V #PWR3
 U 1 1 57C33EC3
 P 4250 1200
-F 0 "#PWR05" H 4250 1050 50  0001 C CNN
+F 0 "#PWR3" H 4250 1050 50  0001 C CNN
 F 1 "+5V" H 4250 1340 50  0000 C CNN
 F 2 "" H 4250 1200 50  0000 C CNN
@@
 $EndComp
 $Comp
-L GND #PWR06
+L GND #PWR4
 U 1 1 57C33F05
 P 4250 1500
-F 0 "#PWR06" H 4250 1250 50  0001 C CNN
+F 0 "#PWR4" H 4250 1250 50  0001 C CNN
 F 1 "GND" H 4250 1350 50  0000 C CNN
 F 2 "" H 4250 1500 50  0000 C CNN
@@
 	1    0    0    1
 $EndComp
-Text GLabel 1550 1550 2    60   Input ~ 0
+Text GLabel 2500 1550 2    60   Input ~ 0
 AC-live-out
-Text GLabel 2500 1250 2    60   Input ~ 0
+Text GLabel 2500 1200 2    60   Input ~ 0
 AC-neut
 $Comp
@@
 	-1   0    0    1
 $EndComp
-Text GLabel 2300 2050 2    60   Input ~ 0
+Text GLabel 2500 1050 2    60   Input ~ 0
 AC-live-f-low
 $Comp
-L R R?
+L R R11
 U 1 1 57C402C2
-P 2250 1400
-F 0 "R?" V 2330 1400 50  0000 C CNN
-F 1 "R" V 2250 1400 50  0000 C CNN
-F 2 "" V 2180 1400 50  0000 C CNN
-F 3 "" H 2250 1400 50  0000 C CNN
-	1    2250 1400
+P 2250 1350
+F 0 "R11" V 2330 1350 50  0000 C CNN
+F 1 "0" V 2250 1350 50  0000 C CNN
+F 2 "Resistors_ThroughHole:Resistor_Horizontal_RM7mm" V 2180 1350 50  0001 C CNN
+F 3 "" H 2250 1350 50  0000 C CNN
+	1    2250 1350
 	0    1    1    0
 $EndComp
 Wire Wire Line
-	950  2250 1900 2250
+	1550 2250 1900 2250
 Wire Wire Line
 	1800 2250 1800 2700
@@
 Connection ~ 4950 2650
 Wire Wire Line
-	2150 1850 2300 1850
-Wire Wire Line
-	1650 1850 1500 1850
-Wire Wire Line
-	1950 1150 1700 1150
-Wire Wire Line
-	1700 1150 1700 1250
-Wire Wire Line
-	1700 1250 1350 1250
-Wire Wire Line
 	4250 1500 4250 1400
 Wire Wire Line
@@
 	2500 4450 2500 4100
 Wire Wire Line
-	1350 1550 1550 1550
-Wire Wire Line
-	2300 2050 2200 2050
-Wire Wire Line
-	2200 2050 2200 1850
-Connection ~ 2200 1850
-Wire Wire Line
-	2500 1250 1800 1250
-Wire Wire Line
-	1800 1250 1800 1350
-Wire Wire Line
-	1800 1350 1350 1350
-Wire Wire Line
-	1800 1450 1350 1450
-Wire Wire Line
-	1800 1300 1800 1450
-Connection ~ 1800 1450
-Connection ~ 1800 1300
-Wire Wire Line
-	2500 1650 950  1650
-Wire Wire Line
-	950  1650 950  2250
-Wire Wire Line
-	2400 1400 2500 1400
-Wire Wire Line
-	2500 1400 2500 1650
-Wire Wire Line
-	2100 1400 1800 1400
-Connection ~ 1800 1400
+	1350 1550 2500 1550
+Wire Wire Line
+	2500 1200 2000 1200
+Wire Wire Line
+	1350 1350 2100 1350
+Wire Wire Line
+	2400 1350 2500 1350
+Text GLabel 2500 1350 2    60   Input ~ 0
+AC-neut-low
+Text GLabel 1550 2250 0    60   Input ~ 0
+AC-live-f-low
+$Comp
+L R R12
+U 1 1 57C4239E
+P 2250 1050
+F 0 "R12" V 2330 1050 50  0000 C CNN
+F 1 "0" V 2250 1050 50  0000 C CNN
+F 2 "Resistors_ThroughHole:Resistor_Horizontal_RM7mm" V 2180 1050 50  0001 C CNN
+F 3 "" H 2250 1050 50  0000 C CNN
+	1    2250 1050
+	0    1    1    0
+$EndComp
+Wire Wire Line
+	2000 1050 2100 1050
+Wire Wire Line
+	2000 1200 2000 1450
+Connection ~ 2000 1350
+Wire Wire Line
+	2400 1050 2500 1050
+Wire Wire Line
+	1900 900  2500 900
+Wire Wire Line
+	2000 900  2000 1050
+Connection ~ 2000 1050
+Connection ~ 2000 900
+Wire Wire Line
+	2000 1450 1350 1450
+Wire Wire Line
+	1400 900  1350 900
+Wire Wire Line
+	1350 900  1350 1250
 $EndSCHEMATC

Commit message: update
Parts:
- added R?: 0, Resistors_ThroughHole:Resistor_Horizontal_RM7mm, symbol R
Connections:
- net labels added: Earth, earth
- wire segments 64 -> 94
Changed lines of the file:
@@
 $EndComp
 $Comp
-L GND #PWR6
+L GND #PWR01
 U 1 1 57C1A76B
 P 4950 3750
-F 0 "#PWR6" H 4950 3500 50  0001 C CNN
+F 0 "#PWR01" H 4950 3500 50  0001 C CNN
 F 1 "GND" H 4950 3600 50  0000 C CNN
 F 2 "" H 4950 3750 50  0000 C CNN
@@
 $EndComp
 $Comp
-L +5V #PWR5
+L +5V #PWR02
 U 1 1 57C1A7D8
 P 4950 2450
-F 0 "#PWR5" H 4950 2300 50  0001 C CNN
+F 0 "#PWR02" H 4950 2300 50  0001 C CNN
 F 1 "+5V" H 4950 2590 50  0000 C CNN
 F 2 "" H 4950 2450 50  0000 C CNN
@@
 $EndComp
 $Comp
-L +5V #PWR1
+L +5V #PWR03
 U 1 1 57C1B997
 P 1150 3550
-F 0 "#PWR1" H 1150 3400 50  0001 C CNN
+F 0 "#PWR03" H 1150 3400 50  0001 C CNN
 F 1 "+5V" H 1150 3690 50  0000 C CNN
 F 2 "" H 1150 3550 50  0000 C CNN
@@
 $EndComp
 $Comp
-L GND #PWR2
+L GND #PWR04
 U 1 1 57C1BA06
 P 1150 5500
-F 0 "#PWR2" H 1150 5250 50  0001 C CNN
+F 0 "#PWR04" H 1150 5250 50  0001 C CNN
 F 1 "GND" H 1150 5350 50  0000 C CNN
 F 2 "" H 1150 5500 50  0000 C CNN
@@
 AC-live-out
 $Comp
-L +5V #PWR3
+L +5V #PWR05
 U 1 1 57C33EC3
 P 4250 1200
-F 0 "#PWR3" H 4250 1050 50  0001 C CNN
+F 0 "#PWR05" H 4250 1050 50  0001 C CNN
 F 1 "+5V" H 4250 1340 50  0000 C CNN
 F 2 "" H 4250 1200 50  0000 C CNN
@@
 $EndComp
 $Comp
-L GND #PWR4
+L GND #PWR06
 U 1 1 57C33F05
 P 4250 1500
-F 0 "#PWR4" H 4250 1250 50  0001 C CNN
+F 0 "#PWR06" H 4250 1250 50  0001 C CNN
 F 1 "GND" H 4250 1350 50  0000 C CNN
 F 2 "" H 4250 1500 50  0000 C CNN
@@
 $EndComp
 Wire Wire Line
-	1550 2250 1900 2250
+	1550 2250 1800 2250
+Wire Wire Line
+	1800 2250 1900 2250
 Wire Wire Line
 	1800 2250 1800 2700
@@
 Connection ~ 1800 2250
 Wire Wire Line
-	2200 2250 3000 2250
+	2200 2250 2350 2250
+Wire Wire Line
+	2350 2250 3000 2250
 Wire Wire Line
 	2200 2700 2350 2700
@@
 	3000 2250 3000 2450
 Wire Wire Line
-	2950 2450 3050 2450
+	2950 2450 3000 2450
+Wire Wire Line
+	3000 2450 3050 2450
 Connection ~ 3000 2450
 Wire Wire Line
-	2650 2450 2650 2850
-Wire Wire Line
-	3350 2450 3350 2850
-Wire Wire Line
-	2950 2850 3050 2850
+	2650 2450 2650 2650
+Wire Wire Line
+	2650 2650 2650 2850
+Wire Wire Line
+	3350 2450 3350 2650
+Wire Wire Line
+	3350 2650 3350 2850
+Wire Wire Line
+	2950 2850 3000 2850
+Wire Wire Line
+	3000 2850 3050 2850
 Wire Wire Line
 	3000 3050 3000 2850
@@
 Connection ~ 2650 2650
 Wire Wire Line
-	3350 2650 4950 2650
+	3350 2650 3750 2650
+Wire Wire Line
+	3750 2650 4400 2650
+Wire Wire Line
+	4400 2650 4950 2650
 Connection ~ 3350 2650
 Wire Wire Line
@@
 Connection ~ 3750 2650
 Wire Wire Line
-	4400 3050 4400 3150
-Wire Wire Line
-	2500 3550 4950 3550
+	4400 3050 4400 3100
+Wire Wire Line
+	4400 3100 4400 3150
+Wire Wire Line
+	2500 3550 3750 3550
+Wire Wire Line
+	3750 3550 4400 3550
+Wire Wire Line
+	4400 3550 4950 3550
 Wire Wire Line
 	4400 3100 4650 3100
@@
 Connection ~ 4400 2650
 Wire Wire Line
-	4950 3300 4950 3750
+	4950 3300 4950 3550
+Wire Wire Line
+	4950 3550 4950 3750
 Wire Wire Line
 	3750 3550 3750 3200
@@
 	3300 4750 3400 4750
 Wire Wire Line
-	1150 4100 4750 4100
-Wire Wire Line
-	1750 4500 1750 4950
+	1150 4100 1750 4100
+Wire Wire Line
+	1750 4100 2500 4100
+Wire Wire Line
+	2500 4100 4750 4100
+Wire Wire Line
+	1750 4500 1750 4850
+Wire Wire Line
+	1750 4850 1750 4950
 Wire Wire Line
 	2300 4850 1750 4850
@@
 	1750 5350 1750 5250
 Wire Wire Line
-	1150 5350 3700 5350
+	1150 5350 1450 5350
+Wire Wire Line
+	1450 5350 1750 5350
+Wire Wire Line
+	1750 5350 2500 5350
+Wire Wire Line
+	2500 5350 3700 5350
 Connection ~ 2500 5350
 Wire Wire Line
-	1150 4000 1150 4200
+	1150 4000 1150 4100
+Wire Wire Line
+	1150 4100 1150 4200
 Connection ~ 1750 4100
 Wire Wire Line
-	1150 4500 1150 4950
-Wire Wire Line
-	1150 5250 1150 5500
+	1150 4500 1150 4650
+Wire Wire Line
+	1150 4650 1150 4950
+Wire Wire Line
+	1150 5250 1150 5350
+Wire Wire Line
+	1150 5350 1150 5500
 Connection ~ 1750 5350
 Connection ~ 1150 5350
 Wire Wire Line
-	1150 4650 2300 4650
+	1150 4650 1450 4650
+Wire Wire Line
+	1450 4650 2300 4650
 Connection ~ 1150 4650
 Connection ~ 2500 4100
@@
 	4750 4400 4600 4400
 Wire Wire Line
-	5550 4300 6450 4300
+	5550 4300 6200 4300
+Wire Wire Line
+	6200 4300 6450 4300
 Wire Wire Line
 	5550 4500 5700 4500
 Wire Wire Line
-	4950 2450 4950 2900
+	4950 2450 4950 2650
+Wire Wire Line
+	4950 2650 4950 2900
 Connection ~ 4950 2650
 Wire Wire Line
@@
 	2500 1200 2000 1200
 Wire Wire Line
-	1350 1350 2100 1350
+	1350 1350 2000 1350
+Wire Wire Line
+	2000 1350 2100 1350
 Wire Wire Line
 	2400 1350 2500 1350
@@
 	2000 1050 2100 1050
 Wire Wire Line
-	2000 1200 2000 1450
+	2000 1200 2000 1350
+Wire Wire Line
+	2000 1350 2000 1450
 Connection ~ 2000 1350
 Wire Wire Line
 	2400 1050 2500 1050
 Wire Wire Line
-	1900 900  2500 900
+	1900 900  2000 900
+Wire Wire Line
+	2000 900  2500 900
 Wire Wire Line
 	2000 900  2000 1050
@@
 Wire Wire Line
 	1350 900  1350 1250
+$Comp
+L Earth #PWR07
+U 1 1 57C44B9E
+P 5500 1100
+F 0 "#PWR07" H 5500 850 50  0001 C CNN
+F 1 "Earth" H 5500 950 50  0001 C CNN
+F 2 "" H 5500 1100 50  0000 C CNN
+F 3 "" H 5500 1100 50  0000 C CNN
+	1    5500 1100
+	1    0    0    -1
+$EndComp
+Text GLabel 4950 1000 0    60   Input ~ 0
+earth
+Wire Wire Line
+	4950 1000 5100 1000
+$Comp
+L R R?
+U 1 1 57C45714
+P 5250 1000
+F 0 "R?" V 5330 1000 50  0000 C CNN
+F 1 "0" V 5250 1000 50  0000 C CNN
+F 2 "Resistors_ThroughHole:Resistor_Horizontal_RM7mm" V 5180 1000 50  0001 C CNN
+F 3 "" H 5250 1000 50  0000 C CNN
+	1    5250 1000
+	0    1    1    0
+$EndComp
+Wire Wire Line
+	5400 1000 5500 1000
+Wire Wire Line
+	5500 1000 5500 1100
 $EndSCHEMATC

Commit message: with fills
Parts:
- removed R?: 0, Resistors_ThroughHole:Resistor_Horizontal_RM7mm, symbol R
Connections:
- net labels removed: earth
- wire segments 94 -> 93
Changed lines of the file:
@@
 	1    0    0    -1
 $EndComp
-Text GLabel 4950 1000 0    60   Input ~ 0
-earth
 Wire Wire Line
-	4950 1000 5100 1000
-$Comp
-L R R?
-U 1 1 57C45714
-P 5250 1000
-F 0 "R?" V 5330 1000 50  0000 C CNN
-F 1 "0" V 5250 1000 50  0000 C CNN
-F 2 "Resistors_ThroughHole:Resistor_Horizontal_RM7mm" V 5180 1000 50  0001 C CNN
-F 3 "" H 5250 1000 50  0000 C CNN
-	1    5250 1000
-	0    1    1    0
-$EndComp
+	5650 1050 5500 1050
 Wire Wire Line
-	5400 1000 5500 1000
-Wire Wire Line
-	5500 1000 5500 1100
+	5500 1050 5500 1100
 $EndSCHEMATC
