File: inrush-limiter/main.kicad_pcb (KiCad board)
At the start: 2 copper layers, 24 parts, among them K1 RELAY_2RT, P1 CONN_01X06, Q1 PN2222A, Q2 PN2222A, U1 LM393

Commit message: update
Parts:
- moved R10 67.9 mm to (186.7, 95.2), turned to 90 degrees
- moved K1 2.54 mm to (177.8, 94.0)
Connections:
- K1 pad 11: (no net) -> Net-(K1-Pad11)
- K1 pad 21: (no net) -> AC-live-f
- K1 pad 22: (no net) -> Net-(K1-Pad22)
- K1 pad 24: (no net) -> AC-live-out
- K1 pad A1: (no net) -> Net-(K1-PadA1)
- K1 pad A2: (no net) -> Net-(K1-PadA2)
- Q1 pad 3: Net-(K1-Pad8) -> Net-(K1-PadA1)
- R1 pad 2: Net-(K1-Pad9) -> Net-(K1-PadA2)
- R10 pad 1: Net-(K1-Pad3) -> Net-(K1-Pad22)
- R2 pad 1: Net-(K1-Pad9) -> Net-(K1-PadA2)
- R4 pad 1: Net-(K1-Pad9) -> Net-(K1-PadA2)
- U1 pad 8: Net-(K1-Pad9) -> Net-(K1-PadA2)
Routing:
- net Net-(K1-PadA2): track 0.00 -> 81.7 mm
- net Net-(K1-Pad9): track 29.7 -> 0.00 mm
- net Net-(K1-Pad22): track 0.00 -> 25.4 mm
- net GND: track 185.5 -> 209.4 mm
- net Net-(K1-PadA1): track 0.00 -> 15.9 mm

Commit message: update
Parts:
- moved Q1 11.7 mm to (153.7, 86.4), turned to 0 degrees
- moved K1 8.89 mm to (168.9, 94.0)
- moved R10 8.89 mm to (177.8, 95.2)
- moved R9 3.81 mm to (154.9, 59.7)
- moved R8 1.27 mm to (156.2, 80.0)
Routing:
- net AC-live-f: track 33.5 -> 105.6 mm
- net GND: track 209.4 -> 186.3 mm
- net Net-(K1-PadA2): track 81.7 -> 68.7 mm
- net AC-live-out: track 0.00 -> 9.58 mm
- net Net-(K1-PadA1): track 15.9 -> 11.7 mm
- net Net-(Q1-Pad2): track 5.08 -> 6.90 mm
- net Net-(D5-Pad2): track 18.8 -> 20.1 mm
- net Net-(R8-Pad2): track 34.6 -> 34.1 mm

Commit message: update
Parts:
- moved C1 3.81 mm to (118.1, 88.9)
- moved R9 2.54 mm to (154.9, 57.1)
- moved Q1 1.27 mm to (152.4, 86.4)
Routing:
- net Net-(C2-Pad1): track 32.9 -> 23.9 mm
- net Net-(K1-PadA2): track 68.7 -> 65.0 mm
- net Net-(C1-Pad1): track 30.6 -> 27.5 mm
- net GND: track 186.3 -> 188.2 mm
- net Net-(D5-Pad2): track 20.1 -> 18.3 mm
- net Net-(K1-PadA1): track 11.7 -> 13.0 mm
- net Net-(R8-Pad2): track 34.1 -> 33.3 mm
- net Net-(K1-Pad22): track 25.4 -> 24.7 mm
- net Net-(Q1-Pad2): track 6.90 -> 7.45 mm
Other:
- board text removed: "Hi Voltage"

Commit message: ok
Parts:
- added P2: CONN_01X02, Pin_Headers:Pin_Header_Straight_1x02, F.Cu at (120.7, 63.5)
- added P3: CONN_01X02, Pin_Headers:Pin_Header_Straight_1x02, F.Cu at (186.7, 69.8)
- P1: value CONN_01X06 -> CONN_01X02; footprint Pin_Headers:Pin_Header_Straight_1x06 -> Pin_Headers:Pin_Header_Straight_1x02
- moved P1 78.3 mm to (186.7, 45.7)
- moved F1 59.7 mm to (177.8, 53.3)
- moved R7 24.2 mm to (147.3, 68.6), turned to 0 degrees
- moved R1 9.92 mm to (119.4, 69.8), turned to 270 degrees
- moved C2 2.54 mm to (133.3, 57.1)
- moved R6 2.54 mm to (127.0, 49.5)
Connections:
- P1 pad 1: GND -> AC-neut
- P1 pad 2: +5V -> AC-live
Routing:
- net AC-neut: track 28.5 -> 70.5 mm
- net +5V: track 104.2 -> 73.4 mm
- net Net-(D2-Pad2): track 47.1 -> 17.0 mm
- net GND: track 188.2 -> 171.4 mm
- net AC-live-f: track 105.4 -> 89.3 mm
- net AC-live: track 10.4 -> 1.21 mm
- net AC-live-out: track 9.58 -> 18.6 mm
- net Net-(D5-Pad2): track 18.3 -> 19.4 mm
- net Net-(K1-PadA2): track 65.0 -> 65.5 mm
- net Net-(C2-Pad1): track 23.9 -> 23.4 mm

Commit message: ok
Routing:
- net AC-live: track 1.21 -> 9.85 mm
- net GND: track 171.4 -> 169.7 mm
- removed copper zone on B.Cu, net GND
Changed lines of the file:
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@@
   (general
     (links 44)
-    (no_connects 2)
-    (area 106.68 40.124999 208.18486 97.07099)
+    (no_connects 0)
+    (area 106.68 40.08901 191.848334 96.925001)
     (thickness 1.6)
     (drawings 0)
-    (tracks 143)
+    (tracks 144)
     (zones 0)
     (modules 26)
@@
   (segment (start 127 90.17) (end 133.35 90.17) (width 1) (layer B.Cu) (net 1))
   (segment (start 124.46 83.82) (end 124.46 87.63) (width 1) (layer B.Cu) (net 1) (status 30))
+  (segment (start 118.11 91.4) (end 116.8 91.4) (width 1) (layer B.Cu) (net 2))
+  (segment (start 118.11 73.66) (end 124.46 73.66) (width 1) (layer B.Cu) (net 2))
+  (segment (start 115.57 76.2) (end 118.11 73.66) (width 1) (layer B.Cu) (net 2))
+  (segment (start 115.57 90.17) (end 115.57 76.2) (width 1) (layer B.Cu) (net 2))
+  (segment (start 116.8 91.4) (end 115.57 90.17) (width 1) (layer B.Cu) (net 2))
   (segment (start 143.50746 68.57948) (end 139.69746 68.57948) (width 1) (layer B.Cu) (net 2) (status 30))
   (segment (start 139.69746 68.57948) (end 139.7 68.58202) (width 1) (layer B.Cu) (net 2) (status 30))
@@
   (segment (start 149.86 95.25) (end 137.16 95.25) (width 1) (layer B.Cu) (net 2))
   (segment (start 151.13 93.98) (end 149.86 95.25) (width 1) (layer B.Cu) (net 2))
-  (segment (start 118.11 91.4) (end 115.61 91.4) (width 1) (layer B.Cu) (net 2) (status 10))
-  (segment (start 114.38 85.17) (end 114.3 85.09) (width 1) (layer B.Cu) (net 2))
-  (segment (start 114.38 90.17) (end 114.38 85.17) (width 1) (layer B.Cu) (net 2))
-  (segment (start 115.61 91.4) (end 114.38 90.17) (width 1) (layer B.Cu) (net 2))
   (segment (start 154.94 64.77) (end 151.13 64.77) (width 1) (layer B.Cu) (net 2) (status 10))
   (segment (start 151.13 73.66) (end 151.13 64.77) (width 1) (layer B.Cu) (net 2))
   (segment (start 151.13 73.66) (end 139.7 73.66) (width 1) (layer B.Cu) (net 2))
   (segment (start 139.7 73.66) (end 124.46 73.66) (width 1) (layer B.Cu) (net 2))
-  (segment (start 124.46 73.66) (end 118.11 73.66) (width 1) (layer B.Cu) (net 2))
-  (segment (start 114.3 85.09) (end 114.3 77.47) (width 1) (layer B.Cu) (net 2))
-  (segment (start 118.11 73.66) (end 114.3 77.47) (width 1) (layer B.Cu) (net 2))
   (segment (start 124.46 95.25) (end 119.38 95.25) (width 1) (layer B.Cu) (net 2) (status 10))
   (segment (start 118.11 93.98) (end 118.11 91.4) (width 1) (layer B.Cu) (net 2) (status 20))
@@
   (segment (start 127 41.91) (end 133.11 41.91) (width 1) (layer B.Cu) (net 4) (status 30))
   (segment (start 133.11 41.91) (end 133.35 42.15) (width 1) (layer B.Cu) (net 4) (status 30))
+  (segment (start 151.13 45.72) (end 149.86 44.45) (width 1) (layer B.Cu) (net 5))
+  (segment (start 149.86 44.45) (end 143.50798 44.45) (width 1) (layer B.Cu) (net 5))
+  (segment (start 143.50798 44.45) (end 143.50746 44.44948) (width 1) (layer B.Cu) (net 5))
+  (segment (start 143.50746 44.44948) (end 139.69746 44.44948) (width 1) (layer B.Cu) (net 5))
   (segment (start 119.38 69.85) (end 119.38 68.58) (width 1) (layer B.Cu) (net 5) (status 10))
   (segment (start 119.38 60.96) (end 120.65 60.96) (width 1) (layer B.Cu) (net 5) (status 20))
@@
   (segment (start 152.40052 44.45052) (end 151.13104 45.72) (width 1) (layer B.Cu) (net 5) (status 20))
   (segment (start 151.13104 45.72) (end 151.13 45.72) (width 1) (layer B.Cu) (net 5) (status 30))
-  (segment (start 151.13 45.72) (end 149.85948 44.44948) (width 1) (layer B.Cu) (net 5) (status 10))
-  (segment (start 149.85948 44.44948) (end 139.69746 44.44948) (width 1) (layer B.Cu) (net 5) (status 20))
   (segment (start 143.50746 58.41948) (end 146.04948 58.41948) (width 1) (layer B.Cu) (net 6) (status 10))
   (segment (start 147.32 59.69) (end 147.32 68.58) (width 1) (layer B.Cu) (net 6) (status 20))
@@
   (segment (start 158.75 54.61306) (end 158.75254 54.61052) (width 1) (layer B.Cu) (net 7) (status 30))
   (segment (start 166.37 50.8) (end 167.64 52.07) (width 1) (layer B.Cu) (net 7))
-  (segment (start 178.22926 41.91) (end 177.8 42.33926) (width 1) (layer B.Cu) (net 8) (status 30))
+  (segment (start 186.69 43.18) (end 178.64074 43.18) (width 1) (layer B.Cu) (net 8))
+  (segment (start 178.64074 43.18) (end 177.8 42.33926) (width 1) (layer B.Cu) (net 8))
   (segment (start 177.37074 41.91) (end 177.8 42.33926) (width 1) (layer B.Cu) (net 8) (status 30))
   (segment (start 186.69 69.85) (end 178.20132 69.85) (width 1) (layer B.Cu) (net 11) (status 10))
@@
   (segment (start 170.18 69.85) (end 177.39868 69.85) (width 1) (layer B.Cu) (net 11))
   (segment (start 177.39868 69.85) (end 177.8 70.25132) (width 1) (layer B.Cu) (net 11))
-  (segment (start 186.69 67.31) (end 187.96 67.31) (width 1) (layer B.Cu) (net 12) (status 400000))
+  (segment (start 186.69 67.31) (end 187.96 67.31) (width 1) (layer B.Cu) (net 12))
   (segment (start 158.75 76.2) (end 184.15 76.2) (width 1) (layer B.Cu) (net 12))
   (segment (start 154.94 72.39) (end 158.75 76.2) (width 1) (layer B.Cu) (net 12))
@@
   (segment (start 168.91 78.74) (end 176.53 78.74) (width 1) (layer B.Cu) (net 19) (status 10))
   (segment (start 177.8 80.01) (end 177.8 95.25) (width 1) (layer B.Cu) (net 19) (status 20))
-  (zone (net 2) (net_name GND) (layer B.Cu) (hatch edge 0.508)
-    (connect_pads (clearance 0.508))
-    (min_thickness 0.254)
-    (fill (arc_segments 16) (thermal_gap 0.508) (thermal_bridge_width 0.508))
-    (polygon
-      (pts
-        (xy 106.68 74.93) (xy 106.68 73.66) (xy 107.95 73.66) (xy 106.68 74.93)
-      )
-    )
-  )
 )

Commit message: update
Routing:
- net AC-neut: track 70.5 -> 48.9 mm
- net Net-(K1-Pad22): track 24.7 -> 20.2 mm
Other:
- net class power added: clearance 0.5, trace_width 2.5, via_dia 0.6, via_drill 0.4
Changed lines of the file:
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@@
   (general
     (links 44)
-    (no_connects 0)
-    (area 106.68 40.08901 191.848334 96.925001)
+    (no_connects 1)
+    (area 112.885 39.83901 192.098334 97.175001)
     (thickness 1.6)
     (drawings 0)
-    (tracks 144)
+    (tracks 139)
     (zones 0)
     (modules 26)
@@
     (uvia_drill 0.1)
     (add_net +5V)
-    (add_net AC-live)
-    (add_net AC-live-f)
-    (add_net AC-live-out)
-    (add_net AC-neut)
     (add_net GND)
     (add_net "Net-(C1-Pad1)")
@@
     (add_net "Net-(K1-Pad12)")
     (add_net "Net-(K1-Pad14)")
-    (add_net "Net-(K1-Pad22)")
     (add_net "Net-(K1-PadA1)")
     (add_net "Net-(K1-PadA2)")
@@
     (add_net "Net-(R4-Pad2)")
     (add_net "Net-(R8-Pad2)")
+  )
+  (net_class power ""
+    (clearance 0.5)
+    (trace_width 2.5)
+    (via_dia 0.6)
+    (via_drill 0.4)
+    (uvia_dia 0.3)
+    (uvia_drill 0.1)
+    (add_net AC-live)
+    (add_net AC-live-f)
+    (add_net AC-live-out)
+    (add_net AC-neut)
+    (add_net "Net-(K1-Pad22)")
   )
   (module Capacitors_ThroughHole:C_Radial_D8_L13_P3.8 (layer F.Cu)
@@
   (segment (start 127 90.17) (end 133.35 90.17) (width 1) (layer B.Cu) (net 1))
   (segment (start 124.46 83.82) (end 124.46 87.63) (width 1) (layer B.Cu) (net 1) (status 30))
-  (segment (start 118.11 91.4) (end 116.8 91.4) (width 1) (layer B.Cu) (net 2))
+  (segment (start 118.11 91.4) (end 116.8 91.4) (width 1) (layer B.Cu) (net 2) (status 10))
   (segment (start 118.11 73.66) (end 124.46 73.66) (width 1) (layer B.Cu) (net 2))
   (segment (start 115.57 76.2) (end 118.11 73.66) (width 1) (layer B.Cu) (net 2))
@@
   (segment (start 139.69746 54.60948) (end 139.69746 57.15) (width 1) (layer B.Cu) (net 3) (status 10))
   (segment (start 139.69746 57.15) (end 139.69746 58.41948) (width 1) (layer B.Cu) (net 3) (status 20))
-  (segment (start 170.18 59.26074) (end 170.18 43.18) (width 1) (layer B.Cu) (net 4))
+  (segment (start 170.18 59.26074) (end 170.18 43.18) (width 2.5) (layer B.Cu) (net 4))
   (segment (start 168.91 41.91) (end 133.59 41.91) (width 1) (layer B.Cu) (net 4) (status 20))
-  (segment (start 170.18 43.18) (end 168.91 41.91) (width 1) (layer B.Cu) (net 4))
-  (segment (start 133.59 41.91) (end 133.35 42.15) (width 1) (layer B.Cu) (net 4) (status 30))
-  (segment (start 172.72 59.26074) (end 170.18 59.26074) (width 1) (layer B.Cu) (net 4))
-  (segment (start 170.18 59.26074) (end 168.06926 59.26074) (width 1) (layer B.Cu) (net 4))
-  (segment (start 165.1 69.85) (end 168.91 73.66) (width 1) (layer B.Cu) (net 4) (status 20))
-  (segment (start 165.1 62.23) (end 165.1 69.85) (width 1) (layer B.Cu) (net 4))
-  (segment (start 168.06926 59.26074) (end 165.1 62.23) (width 1) (layer B.Cu) (net 4))
-  (segment (start 172.72 59.26074) (end 177.8 64.34074) (width 1) (layer B.Cu) (net 4) (status 20))
-  (segment (start 133.35 42.15) (end 133.35 41.91) (width 1) (layer B.Cu) (net 4) (status 30))
-  (segment (start 127 41.91) (end 133.11 41.91) (width 1) (layer B.Cu) (net 4) (status 30))
-  (segment (start 133.11 41.91) (end 133.35 42.15) (width 1) (layer B.Cu) (net 4) (status 30))
-  (segment (start 151.13 45.72) (end 149.86 44.45) (width 1) (layer B.Cu) (net 5))
-  (segment (start 149.86 44.45) (end 143.50798 44.45) (width 1) (layer B.Cu) (net 5))
-  (segment (start 143.50798 44.45) (end 143.50746 44.44948) (width 1) (layer B.Cu) (net 5))
-  (segment (start 143.50746 44.44948) (end 139.69746 44.44948) (width 1) (layer B.Cu) (net 5))
+  (segment (start 170.18 43.18) (end 168.91 41.91) (width 2.5) (layer B.Cu) (net 4))
+  (segment (start 133.59 41.91) (end 133.35 42.15) (width 2.5) (layer B.Cu) (net 4) (status 30))
+  (segment (start 172.72 59.26074) (end 170.18 59.26074) (width 2.5) (layer B.Cu) (net 4))
+  (segment (start 170.18 59.26074) (end 168.06926 59.26074) (width 2.5) (layer B.Cu) (net 4))
+  (segment (start 165.1 69.85) (end 168.91 73.66) (width 2.5) (layer B.Cu) (net 4) (status 20))
+  (segment (start 165.1 62.23) (end 165.1 69.85) (width 2.5) (layer B.Cu) (net 4))
+  (segment (start 168.06926 59.26074) (end 165.1 62.23) (width 2.5) (layer B.Cu) (net 4))
+  (segment (start 172.72 59.26074) (end 177.8 64.34074) (width 2.5) (layer B.Cu) (net 4) (status 20))
+  (segment (start 133.35 42.15) (end 133.35 41.91) (width 2.5) (layer B.Cu) (net 4) (status 30))
+  (segment (start 127 41.91) (end 133.11 41.91) (width 2.5) (layer B.Cu) (net 4) (status 30))
+  (segment (start 133.11 41.91) (end 133.35 42.15) (width 2.5) (layer B.Cu) (net 4) (status 30))
+  (segment (start 151.13 45.72) (end 149.86 44.45) (width 1) (layer B.Cu) (net 5) (status 10))
+  (segment (start 149.86 44.45) (end 143.50798 44.45) (width 1) (layer B.Cu) (net 5) (status 20))
+  (segment (start 143.50798 44.45) (end 143.50746 44.44948) (width 1) (layer B.Cu) (net 5) (status 30))
+  (segment (start 143.50746 44.44948) (end 139.69746 44.44948) (width 1) (layer B.Cu) (net 5) (status 30))
   (segment (start 119.38 69.85) (end 119.38 68.58) (width 1) (layer B.Cu) (net 5) (status 10))
   (segment (start 119.38 60.96) (end 120.65 60.96) (width 1) (layer B.Cu) (net 5) (status 20))
@@
   (segment (start 158.75 54.61306) (end 158.75254 54.61052) (width 1) (layer B.Cu) (net 7) (status 30))
   (segment (start 166.37 50.8) (end 167.64 52.07) (width 1) (layer B.Cu) (net 7))
-  (segment (start 186.69 43.18) (end 178.64074 43.18) (width 1) (layer B.Cu) (net 8))
-  (segment (start 178.64074 43.18) (end 177.8 42.33926) (width 1) (layer B.Cu) (net 8))
-  (segment (start 177.37074 41.91) (end 177.8 42.33926) (width 1) (layer B.Cu) (net 8) (status 30))
-  (segment (start 186.69 69.85) (end 178.20132 69.85) (width 1) (layer B.Cu) (net 11) (status 10))
-  (segment (start 178.20132 69.85) (end 177.8 70.25132) (width 1) (layer B.Cu) (net 11))
-  (segment (start 168.91 68.58) (end 170.18 69.85) (width 1) (layer B.Cu) (net 11))
-  (segment (start 170.18 69.85) (end 177.39868 69.85) (width 1) (layer B.Cu) (net 11))
-  (segment (start 177.39868 69.85) (end 177.8 70.25132) (width 1) (layer B.Cu) (net 11))
-  (segment (start 186.69 67.31) (end 187.96 67.31) (width 1) (layer B.Cu) (net 12))
+  (segment (start 186.69 43.18) (end 178.64074 43.18) (width 1) (layer B.Cu) (net 8) (status 30))
+  (segment (start 178.64074 43.18) (end 177.8 42.33926) (width 2.5) (layer B.Cu) (net 8) (status 30))
+  (segment (start 177.37074 41.91) (end 177.8 42.33926) (width 2.5) (layer B.Cu) (net 8) (status 30))
+  (segment (start 186.69 69.85) (end 178.20132 69.85) (width 1) (layer B.Cu) (net 11) (status 30))
+  (segment (start 178.20132 69.85) (end 177.8 70.25132) (width 2.5) (layer B.Cu) (net 11) (status 30))
+  (segment (start 168.91 68.58) (end 170.18 69.85) (width 2.5) (layer B.Cu) (net 11) (status 10))
+  (segment (start 170.18 69.85) (end 177.39868 69.85) (width 2.5) (layer B.Cu) (net 11) (status 20))
+  (segment (start 177.39868 69.85) (end 177.8 70.25132) (width 2.5) (layer B.Cu) (net 11) (status 30))
+  (segment (start 186.69 67.31) (end 187.96 67.31) (width 1) (layer B.Cu) (net 12) (status 10))
   (segment (start 158.75 76.2) (end 184.15 76.2) (width 1) (layer B.Cu) (net 12))
   (segment (start 154.94 72.39) (end 158.75 76.2) (width 1) (layer B.Cu) (net 12))
-  (segment (start 154.94 72.39) (end 154.94 68.58) (width 1) (layer B.Cu) (net 12) (status 10))
-  (segment (start 187.96 74.93) (end 186.69 76.2) (width 1) (layer B.Cu) (net 12))
-  (segment (start 186.69 76.2) (end 184.15 76.2) (width 1) (layer B.Cu) (net 12))
-  (segment (start 189.23 73.66) (end 187.96 74.93) (width 1) (layer B.Cu) (net 12))
+  (segment (start 154.94 72.39) (end 154.94 68.58) (width 2.5) (layer B.Cu) (net 12) (status 20))
+  (segment (start 189.23 73.66) (end 186.69 76.2) (width 2.5) (layer B.Cu) (net 12))
+  (segment (start 186.69 76.2) (end 184.15 76.2) (width 2.5) (layer B.Cu) (net 12))
   (segment (start 189.23 68.58) (end 189.23 73.66) (width 1) (layer B.Cu) (net 12))
   (segment (start 187.96 67.31) (end 189.23 68.58) (width 1) (layer B.Cu) (net 12))
-  (segment (start 186.69 67.31) (end 186.69 67.31) (width 1) (layer B.Cu) (net 12) (status 10))
-  (segment (start 186.69 45.72) (end 186.69 66.04) (width 1) (layer B.Cu) (net 12) (status 10))
-  (segment (start 186.69 66.04) (end 186.69 67.31) (width 1) (layer B.Cu) (net 12) (status 20))
   (segment (start 153.67 86.36) (end 153.67 85.09) (width 1) (layer B.Cu) (net 13) (status 10))
   (segment (start 156.21 82.55) (end 156.21 80.01) (width 1) (layer B.Cu) (net 13) (status 20))
@@
   (segment (start 157.48 86.36) (end 161.29 90.17) (width 1) (layer B.Cu) (net 18))
   (segment (start 160.02 93.98) (end 161.29 93.98) (width 1) (layer B.Cu) (net 18) (status 30))
-  (segment (start 176.53 78.74) (end 177.8 80.01) (width 1) (layer B.Cu) (net 19))
-  (segment (start 168.91 78.74) (end 176.53 78.74) (width 1) (layer B.Cu) (net 19) (status 10))
-  (segment (start 177.8 80.01) (end 177.8 95.25) (width 1) (layer B.Cu) (net 19) (status 20))
+  (segment (start 168.91 78.74) (end 177.8 87.63) (width 2.5) (layer B.Cu) (net 19) (status 10))
+  (segment (start 177.8 87.63) (end 177.8 95.25) (width 2.5) (layer B.Cu) (net 19) (status 20))
 )

Commit message: update
Parts:
- removed P3: CONN_01X02, Pin_Headers:Pin_Header_Straight_1x02
- P1: value CONN_01X02 -> CONN_01X04; footprint Pin_Headers:Pin_Header_Straight_1x02 -> Connect:AK300-4
- moved P1 14.9 mm to (191.8, 59.7), turned to 90 degrees
Connections:
- P1 pad 1: AC-neut -> AC-live-out
- P1 pad 2: AC-live -> AC-neut
Routing:
- net AC-neut: track 48.9 -> 5.00 mm
- net AC-live-out: track 18.6 -> 29.1 mm
- net AC-live: track 9.85 -> 14.9 mm
- net GND: track 169.7 -> 171.7 mm
- net AC-live-f: track 89.3 -> 90.3 mm
Other:
- net class power: trace_width 2.5 -> 3

Commit message: update
Connections:
- K1 pad 11: Net-(K1-Pad11) -> (no net)
- K1 pad 12: Net-(K1-Pad12) -> (no net)
- K1 pad 14: Net-(K1-Pad14) -> (no net)
Routing:
- net AC-live-f: track 90.3 -> 23.3 mm
- net AC-neut: track 5.00 -> 0.00 mm
