File: inrush-limiter2/main.sch (KiCad schematic (older format))
At the start: 37 parts, among them K1 RELAY_2RT, P1 CONN_01X04, Q2 PN2222A

Commit message: update
Parts:
- removed R10: 100, 5W, Resistors_ThroughHole:Resistor_Horizontal_RM25mm, symbol R
- added 1M: RVAR, symbol RVAR
- added 1k, R?: R, symbol R
- added 470nF: CP, symbol CP
- added Q?: 2N3904, symbol 2N3904
- added U?: LM393, symbol LM393
Connections:
- wire segments 86 -> 96
Other:
- moved on the sheet: 10k, 5k, C?, K1, Q?

Commit message: update
Parts:
- removed 10k (x2), 5k, R?: R, symbol R
- removed C?: CP, symbol CP
- removed D5: ZENER, Diodes_ThroughHole:Diode_DO-35_SOD27_Horizontal_RM10, symbol ZENER
- removed D6: LED, LEDs:LED-5MM, symbol LED
- removed Q2: PN2222A, TO_SOT_Packages_THT:TO-92_Inline_Wide, symbol PN2222A
- removed Q? (x2): 2N3904, symbol 2N3904
- removed Q?: 2N3906, symbol 2N3906
- removed R13: 140, Resistors_ThroughHole:Resistor_Horizontal_RM7mm, symbol R
- removed R9: 2k, Resistors_ThroughHole:Resistor_Horizontal_RM7mm, symbol R
- gave numbers to parts that had none: 1
Connections:
- net labels removed: Earth
- wire segments 96 -> 95
Other:
- moved on the sheet: 100k, 10k, 1M, 1k, 470nF, D7, K1, Q?, R14, U?A

Commit message: update
Parts:
- removed C2: 47nF, x2, Capacitors_ThroughHole:C_Rect_L18_W5_P15, symbol C
- removed R6: 470k, Resistors_ThroughHole:Resistor_Horizontal_RM7mm, symbol R
- removed R7: 100, Resistors_ThroughHole:Resistor_Horizontal_RM7mm, symbol R
- added D?: LED, symbol LED
- added R?: R, symbol R
- added T?: TRANSFO, symbol TRANSFO
- renumbered 1k to 2k
Connections:
- wire segments 95 -> 72
Other:
- moved on the sheet: 10k, 1k, 470nF, C3, D1, D2, D3, D4, D7, K1, Q?, U?A

Commit message: update
Parts:
- added 100: R, symbol R
Connections:
- wire segments 72 -> 76
Changed lines of the file:
@@
 Wire Wire Line
 	4700 3400 4700 3600
+Text GLabel 8850 4250 2    60   Input ~ 0
+AC-live-f
+$Comp
+L R 100
+U 1 1 57CC96A4
+P 8450 4450
+F 0 "100 ohm NTC" V 8530 4450 50  0000 C CNN
+F 1 "R" V 8450 4450 50  0000 C CNN
+F 2 "" V 8380 4450 50  0000 C CNN
+F 3 "" H 8450 4450 50  0000 C CNN
+	1    8450 4450
+	0    1    1    0
+$EndComp
+Wire Wire Line
+	8850 4250 8100 4250
+Wire Wire Line
+	8700 4250 8700 4450
+Wire Wire Line
+	8700 4450 8600 4450
+Connection ~ 8700 4250
+Wire Wire Line
+	8300 4450 8100 4450
 $EndSCHEMATC

Commit message: update
Parts:
- added U?: LM393, symbol LM393
Connections:
- wire segments 76 -> 83
Changed lines of the file:
@@
 Wire Wire Line
 	8300 4450 8100 4450
+$Comp
+L LM393 U?
+U 2 1 57CCA21B
+P 5550 6300
+F 0 "U?" H 5700 6450 50  0000 C CNN
+F 1 "LM393" H 5800 6150 50  0000 C CNN
+F 2 "" H 5550 6300 50  0000 C CNN
+F 3 "" H 5550 6300 50  0000 C CNN
+	2    5550 6300
+	1    0    0    -1
+$EndComp
+Wire Wire Line
+	5250 6200 4950 6200
+Wire Wire Line
+	4950 6200 4950 6700
+Wire Wire Line
+	4950 6400 5250 6400
+Wire Wire Line
+	4950 6700 6000 6700
+Wire Wire Line
+	6000 6700 6000 6300
+Wire Wire Line
+	6000 6300 5850 6300
+Connection ~ 4950 6400
+Wire Wire Line
+	5450 6600 5450 6700
+Connection ~ 5450 6700
 $EndSCHEMATC

Commit message: update
Parts:
- added MOV: R, symbol R
Connections:
- wire segments 83 -> 117
Other:
- moved on the sheet: 100 ohm NTC, 100k, 10k, 1M, 1k, 2k, 470nF, 5.6V, C3, D1, D2, D3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

Commit message: update and add cache files
Parts:
- removed R1: 0, Resistors_ThroughHole:Resistor_Horizontal_RM7mm, symbol R
- added 0: R, symbol R
- renumbered 100 to 100~ohm~NTC
Connections:
- wire segments 117 -> 119
Other:
- moved on the sheet: 1M, C3, U?B
Changed lines of the file:
@@
 L CP C3
 U 1 1 57C0C56F
-P 4350 2800
-F 0 "C3" H 4375 2900 50  0000 L CNN
-F 1 "100uF, 25V" H 4375 2700 50  0000 L CNN
-F 2 "Capacitors_ThroughHole:C_Radial_D8_L13_P3.8" H 4388 2650 50  0001 C CNN
-F 3 "" H 4350 2800 50  0000 C CNN
-	1    4350 2800
+P 4350 2950
+F 0 "C3" H 4375 3050 50  0000 L CNN
+F 1 "100uF, 25V" H 4375 2850 50  0000 L CNN
+F 2 "Capacitors_ThroughHole:C_Radial_D8_L13_P3.8" H 4388 2800 50  0001 C CNN
+F 3 "" H 4350 2950 50  0000 C CNN
+	1    4350 2950
 	1    0    0    -1
 $EndComp
@@
 L +5V #PWR01
 U 1 1 57C1B997
-P 1150 3750
-F 0 "#PWR01" H 1150 3600 50  0001 C CNN
-F 1 "+5V" H 1150 3890 50  0000 C CNN
-F 2 "" H 1150 3750 50  0000 C CNN
-F 3 "" H 1150 3750 50  0000 C CNN
-	1    1150 3750
+P 1150 4050
+F 0 "#PWR01" H 1150 3900 50  0001 C CNN
+F 1 "+5V" H 1150 4190 50  0000 C CNN
+F 2 "" H 1150 4050 50  0000 C CNN
+F 3 "" H 1150 4050 50  0000 C CNN
+	1    1150 4050
 	1    0    0    -1
 $EndComp
@@
 Text GLabel 5600 5550 2    60   Input ~ 0
 AC-live-out
-$Comp
-L R R1
-U 1 1 57C35DF4
-P 1150 4000
-F 0 "R1" V 1230 4000 50  0000 C CNN
-F 1 "0" V 1150 4000 50  0000 C CNN
-F 2 "Resistors_ThroughHole:Resistor_Horizontal_RM7mm" V 1080 4000 50  0001 C CNN
-F 3 "" H 1150 4000 50  0000 C CNN
-	1    1150 4000
-	1    0    0    -1
-$EndComp
 $Comp
 L RELAY_2RT K1
@@
 L RVAR 1M
 U 1 1 57CC0108
-P 2700 4900
-F 0 "1M" V 2780 4850 50  0000 C CNN
-F 1 "RVAR" V 2620 4960 50  0000 C CNN
-F 2 "" H 2700 4900 50  0000 C CNN
-F 3 "" H 2700 4900 50  0000 C CNN
-	1    2700 4900
+P 2650 4900
+F 0 "1M" V 2730 4850 50  0000 C CNN
+F 1 "RVAR" V 2570 4960 50  0000 C CNN
+F 2 "" H 2650 4900 50  0000 C CNN
+F 3 "" H 2650 4900 50  0000 C CNN
+	1    2650 4900
 	0    1    1    0
 $EndComp
@@
 AC-live-f
 $Comp
-L R 100
+L R 100~ohm~NTC
 U 1 1 57CC96A4
 P 6800 4750
@@
 L LM393 U?
 U 2 1 57CCA21B
-P 3850 6500
-F 0 "U?" H 4000 6650 50  0000 C CNN
-F 1 "LM393" H 4100 6350 50  0000 C CNN
-F 2 "" H 3850 6500 50  0000 C CNN
-F 3 "" H 3850 6500 50  0000 C CNN
-	2    3850 6500
+P 3850 6700
+F 0 "U?" H 4000 6850 50  0000 C CNN
+F 1 "LM393" H 4100 6550 50  0000 C CNN
+F 2 "" H 3850 6700 50  0000 C CNN
+F 3 "" H 3850 6700 50  0000 C CNN
+	2    3850 6700
 	1    0    0    -1
 $EndComp
@@
 Wire Wire Line
 	1350 1450 1350 1400
-Connection ~ 3750 6900
-Wire Wire Line
-	3750 6900 3750 6800
-Connection ~ 3250 6600
-Wire Wire Line
-	3250 6900 3750 6900
-Wire Wire Line
-	3250 6600 3550 6600
-Wire Wire Line
-	3250 6400 3250 6600
-Wire Wire Line
-	3250 6600 3250 6900
-Wire Wire Line
-	3550 6400 3250 6400
+Connection ~ 3750 7100
+Wire Wire Line
+	3750 7000 3750 7100
+Wire Wire Line
+	3750 7100 3750 7450
+Connection ~ 3250 6800
+Wire Wire Line
+	3250 7100 3750 7100
+Wire Wire Line
+	3250 6800 3550 6800
+Wire Wire Line
+	3250 6600 3250 6800
+Wire Wire Line
+	3250 6800 3250 7100
+Wire Wire Line
+	3550 6600 3250 6600
 Wire Wire Line
 	6650 4750 6450 4750
@@
 	1150 5900 1150 6200
 Wire Wire Line
-	1150 4150 1150 4350
+	1150 4000 1150 4350
 Wire Wire Line
 	1150 4350 1150 4700
@@
 Connection ~ 2250 4900
 Wire Wire Line
-	2450 4900 2250 4900
+	2400 4900 2250 4900
 Wire Wire Line
 	2250 4800 2250 4900
@@
 	1350 1550 3900 1550
 Wire Wire Line
-	1150 3700 1150 3850
-Wire Wire Line
 	1150 4350 1600 4350
 Wire Wire Line
@@
 Wire Wire Line
 	4950 4350 5650 4350
-Wire Wire Line
-	6000 2400 6550 2400
 Wire Wire Line
 	2800 2800 3600 2800
 Connection ~ 4350 2400
 Wire Wire Line
-	4350 2400 4350 2650
+	4350 2400 4350 2800
 Connection ~ 3950 2400
 Wire Wire Line
@@
 Wire Wire Line
 	3100 2400 3100 3650
+$Comp
+L GND #PWR?
+U 1 1 57CE7D0C
+P 3750 7500
+F 0 "#PWR?" H 3750 7250 50  0001 C CNN
+F 1 "GND" H 3750 7350 50  0000 C CNN
+F 2 "" H 3750 7500 50  0000 C CNN
+F 3 "" H 3750 7500 50  0000 C CNN
+	1    3750 7500
+	1    0    0    -1
+$EndComp
+$Comp
+L R 0
+U 1 1 57CE8283
+P 6300 2400
+F 0 "0 ohm" V 6380 2400 50  0000 C CNN
+F 1 "R" V 6300 2400 50  0000 C CNN
+F 2 "" V 6230 2400 50  0000 C CNN
+F 3 "" H 6300 2400 50  0000 C CNN
+	1    6300 2400
+	0    1    1    0
+$EndComp
+Wire Wire Line
+	6000 2400 6150 2400
+Wire Wire Line
+	6450 2400 6550 2400
+Wire Wire Line
+	3750 6200 3750 6400
+$Comp
+L +5V #PWR?
+U 1 1 57CE86AC
+P 3750 6200
+F 0 "#PWR?" H 3750 6050 50  0001 C CNN
+F 1 "+5V" H 3750 6340 50  0000 C CNN
+F 2 "" H 3750 6200 50  0000 C CNN
+F 3 "" H 3750 6200 50  0000 C CNN
+	1    3750 6200
+	1    0    0    -1
+$EndComp
 $EndSCHEMATC

Commit message: update
Parts:
- CP: renamed from 470nF; value CP -> 470nF
- D: renamed from 5.6V; value ZENER -> 5.6V
- MOV?: renamed from MOV; value R -> MOV
- R: renamed from 2k; value R -> 2k
- R, R?: renamed from 100k; value R -> 100k
- R: renamed from 10k; value R -> 10k
- R: renamed from 1k; value R -> 2k
- R: renamed from R?; value R -> 140
- R: renamed from 0; value R -> 0
- RVAR: renamed from 1M; value RVAR -> 1M
- U?: renamed from 100~ohm~NTC; value R -> 50 ohm NTC
- renumbered C3 to C?, D1 to D?, D3 to D?, D2 to D?, D4 to D?, D7 to D?, F1 to F?, K1 to K?, P1 to P?, R14 to R, R11 to R?, R12 to R?
Connections:
- wire segments 119 -> 118
Changed lines of the file:
@@
 $EndDescr
 $Comp
-L FUSE F1
+L FUSE F?
 U 1 1 57C0C016
 P 1950 750
-F 0 "F1" H 2050 800 50  0000 C CNN
+F 0 "F?" H 2050 800 50  0000 C CNN
 F 1 "FUSE" H 1850 700 50  0000 C CNN
 F 2 "Fuse_Holders_and_Fuses:Fuseholder5x20_horiz_SemiClosed_Casing10x25mm" H 1950 750 50  0001 C CNN
@@
 $EndComp
 $Comp
-L 1N4007 D1
+L 1N4007 D?
 U 1 1 57C0C128
 P 3400 2200
-F 0 "D1" H 3400 2300 50  0000 C CNN
+F 0 "D?" H 3400 2300 50  0000 C CNN
 F 1 "D" H 3400 2100 50  0000 C CNN
 F 2 "Diodes_ThroughHole:Diode_DO-35_SOD27_Horizontal_RM10" H 3400 2200 50  0001 C CNN
@@
 $EndComp
 $Comp
-L 1N4007 D3
+L 1N4007 D?
 U 1 1 57C0C217
 P 3800 2200
-F 0 "D3" H 3800 2300 50  0000 C CNN
+F 0 "D?" H 3800 2300 50  0000 C CNN
 F 1 "D" H 3800 2100 50  0000 C CNN
 F 2 "Diodes_ThroughHole:Diode_DO-35_SOD27_Horizontal_RM10" H 3800 2200 50  0001 C CNN
@@
 $EndComp
 $Comp
-L 1N4007 D2
+L 1N4007 D?
 U 1 1 57C0C23E
 P 3400 2600
-F 0 "D2" H 3400 2700 50  0000 C CNN
+F 0 "D?" H 3400 2700 50  0000 C CNN
 F 1 "D" H 3400 2500 50  0000 C CNN
 F 2 "Diodes_ThroughHole:Diode_DO-35_SOD27_Horizontal_RM10" H 3400 2600 50  0001 C CNN
@@
 $EndComp
 $Comp
-L 1N4007 D4
+L 1N4007 D?
 U 1 1 57C0C26B
 P 3800 2600
-F 0 "D4" H 3800 2700 50  0000 C CNN
+F 0 "D?" H 3800 2700 50  0000 C CNN
 F 1 "D" H 3800 2500 50  0000 C CNN
 F 2 "Diodes_ThroughHole:Diode_DO-35_SOD27_Horizontal_RM10" H 3800 2600 50  0001 C CNN
@@
 $EndComp
 $Comp
-L CP C3
+L CP C?
 U 1 1 57C0C56F
 P 4350 2950
-F 0 "C3" H 4375 3050 50  0000 L CNN
+F 0 "C?" H 4375 3050 50  0000 L CNN
 F 1 "100uF, 25V" H 4375 2850 50  0000 L CNN
 F 2 "Capacitors_ThroughHole:C_Radial_D8_L13_P3.8" H 4388 2800 50  0001 C CNN
@@
 $EndComp
 $Comp
-L +5V #PWR01
+L +5V #PWR?
 U 1 1 57C1B997
 P 1150 4050
-F 0 "#PWR01" H 1150 3900 50  0001 C CNN
+F 0 "#PWR?" H 1150 3900 50  0001 C CNN
 F 1 "+5V" H 1150 4190 50  0000 C CNN
 F 2 "" H 1150 4050 50  0000 C CNN
@@
 $EndComp
 $Comp
-L GND #PWR02
+L GND #PWR?
 U 1 1 57C1BA06
 P 1150 6200
-F 0 "#PWR02" H 1150 5950 50  0001 C CNN
+F 0 "#PWR?" H 1150 5950 50  0001 C CNN
 F 1 "GND" H 1150 6050 50  0000 C CNN
 F 2 "" H 1150 6200 50  0000 C CNN
@@
 AC-live-out
 $Comp
-L RELAY_2RT K1
+L RELAY_2RT K?
 U 1 1 57C3B514
 P 6050 4700
-F 0 "K1" H 6000 5100 50  0000 C CNN
+F 0 "K?" H 6000 5100 50  0000 C CNN
 F 1 "RELAY_2RT" H 6200 4200 50  0000 C CNN
 F 2 "Relays_ThroughHole:Relay_DPDT_Schrack-RT2_RM5mm" H 6050 4700 50  0001 C CNN
@@
 AC-neut
 $Comp
-L CONN_01X04 P1
+L CONN_01X04 P?
 U 1 1 57C3EB1A
 P 1150 1400
-F 0 "P1" H 1150 1650 50  0000 C CNN
+F 0 "P?" H 1150 1650 50  0000 C CNN
 F 1 "CONN_01X04" V 1250 1400 50  0000 C CNN
 F 2 "Connect:AK300-4" H 1150 1400 50  0001 C CNN
@@
 AC-live-f-low
 $Comp
-L R R11
+L R R?
 U 1 1 57C402C2
 P 3650 1350
-F 0 "R11" V 3730 1350 50  0000 C CNN
+F 0 "R?" V 3730 1350 50  0000 C CNN
 F 1 "0" V 3650 1350 50  0000 C CNN
 F 2 "Resistors_ThroughHole:Resistor_Horizontal_RM7mm" V 3580 1350 50  0001 C CNN
@@
 AC-live-f-low
 $Comp
-L R R12
+L R R?
 U 1 1 57C4239E
 P 3650 1050
-F 0 "R12" V 3730 1050 50  0000 C CNN
+F 0 "R?" V 3730 1050 50  0000 C CNN
 F 1 "0" V 3650 1050 50  0000 C CNN
 F 2 "Resistors_ThroughHole:Resistor_Horizontal_RM7mm" V 3580 1050 50  0001 C CNN
@@
 $EndComp
 $Comp
-L R R14
+L R R
 U 1 1 57C521F5
 P 1150 4850
-F 0 "R14" V 1230 4850 50  0000 C CNN
+F 0 "R" V 1230 4850 50  0000 C CNN
 F 1 "140" V 1150 4850 50  0000 C CNN
 F 2 "Resistors_ThroughHole:Resistor_Horizontal_RM7mm" V 1080 4850 50  0001 C CNN
@@
 $EndComp
 $Comp
-L LED D7
+L LED D?
 U 1 1 57C53617
 P 1150 5400
-F 0 "D7" H 1150 5500 50  0000 C CNN
+F 0 "D?" H 1150 5500 50  0000 C CNN
 F 1 "LED" H 1150 5300 50  0000 C CNN
 F 2 "LEDs:LED-5MM" H 1150 5400 50  0001 C CNN
@@
 $EndComp
 $Comp
-L ZENER 5.6V
+L ZENER D
 U 1 1 57CB6BB5
 P 5200 3300
-F 0 "5.6V" H 5200 3400 50  0000 C CNN
-F 1 "ZENER" H 5200 3200 50  0000 C CNN
+F 0 "D" H 5200 3400 50  0000 C CNN
+F 1 "5.6V" H 5200 3200 50  0000 C CNN
 F 2 "" H 5200 3300 50  0000 C CNN
 F 3 "" H 5200 3300 50  0000 C CNN
@@
 $EndComp
 $Comp
-L R 2k
+L R R
 U 1 1 57CB6C1C
 P 5200 2750
-F 0 "2k" V 5280 2750 50  0000 C CNN
-F 1 "R" V 5200 2750 50  0000 C CNN
+F 0 "R" V 5280 2750 50  0000 C CNN
+F 1 "2k" V 5200 2750 50  0000 C CNN
 F 2 "" V 5130 2750 50  0000 C CNN
 F 3 "" H 5200 2750 50  0000 C CNN
@@
 $EndComp
 $Comp
-L R 100k
+L R R
 U 1 1 57CB72EE
 P 1600 4750
-F 0 "100k" V 1680 4750 50  0000 C CNN
-F 1 "R" V 1600 4750 50  0000 C CNN
+F 0 "R" V 1680 4750 50  0000 C CNN
+F 1 "100k" V 1600 4750 50  0000 C CNN
 F 2 "" V 1530 4750 50  0000 C CNN
 F 3 "" H 1600 4750 50  0000 C CNN
@@
 $EndComp
 $Comp
-L R 100k
+L R R
 U 1 1 57CB739A
 P 1600 5450
-F 0 "100k" V 1680 5450 50  0000 C CNN
-F 1 "R" V 1600 5450 50  0000 C CNN
+F 0 "R" V 1680 5450 50  0000 C CNN
+F 1 "100k" V 1600 5450 50  0000 C CNN
 F 2 "" V 1530 5450 50  0000 C CNN
 F 3 "" H 1600 5450 50  0000 C CNN
@@
 $EndComp
 $Comp
-L R 100k
+L R R?
 U 1 1 57CB9401
 P 2250 4650
-F 0 "100k" V 2330 4650 50  0000 C CNN
-F 1 "R" V 2250 4650 50  0000 C CNN
+F 0 "R?" V 2330 4650 50  0000 C CNN
+F 1 "100k" V 2250 4650 50  0000 C CNN
 F 2 "" V 2180 4650 50  0000 C CNN
 F 3 "" H 2250 4650 50  0000 C CNN
@@
 $EndComp
 $Comp
-L R 10k
+L R R
 U 1 1 57CB9460
 P 2250 5300
-F 0 "10k" V 2330 5300 50  0000 C CNN
-F 1 "R" V 2250 5300 50  0000 C CNN
+F 0 "R" V 2330 5300 50  0000 C CNN
+F 1 "10k" V 2250 5300 50  0000 C CNN
 F 2 "" V 2180 5300 50  0000 C CNN
 F 3 "" H 2250 5300 50  0000 C CNN
@@
 $EndComp
 $Comp
-L R 100k
+L R R
 U 1 1 57CB94CF
 P 2250 5650
-F 0 "100k" V 2330 5650 50  0000 C CNN
-F 1 "R" V 2250 5650 50  0000 C CNN
+F 0 "R" V 2330 5650 50  0000 C CNN
+F 1 "100k" V 2250 5650 50  0000 C CNN
 F 2 "" V 2180 5650 50  0000 C CNN
 F 3 "" H 2250 5650 50  0000 C CNN
@@
 $EndComp
 $Comp
-L RVAR 1M
+L RVAR RVAR
 U 1 1 57CC0108
 P 2650 4900
-F 0 "1M" V 2730 4850 50  0000 C CNN
-F 1 "RVAR" V 2570 4960 50  0000 C CNN
+F 0 "RVAR" V 2730 4850 50  0000 C CNN
+F 1 "1M" V 2570 4960 50  0000 C CNN
 F 2 "" H 2650 4900 50  0000 C CNN
 F 3 "" H 2650 4900 50  0000 C CNN
@@
 $EndComp
 $Comp
-L CP 470nF
+L CP CP
 U 1 1 57CC0848
 P 3100 5450
-F 0 "470nF" H 3125 5550 50  0000 L CNN
-F 1 "CP" H 3125 5350 50  0000 L CNN
+F 0 "CP" H 3125 5550 50  0000 L CNN
+F 1 "470nF" H 3125 5350 50  0000 L CNN
 F 2 "" H 3138 5300 50  0000 C CNN
 F 3 "" H 3100 5450 50  0000 C CNN
@@
 $EndComp
 $Comp
-L R 1k
+L R R
 U 1 1 57CC12F2
 P 4550 4650
-F 0 "1k" V 4630 4650 50  0000 C CNN
-F 1 "R" V 4550 4650 50  0000 C CNN
+F 0 "R" V 4630 4650 50  0000 C CNN
+F 1 "2k" V 4550 4650 50  0000 C CNN
 F 2 "" V 4480 4650 50  0000 C CNN
 F 3 "" H 4550 4650 50  0000 C CNN
@@
 $EndComp
 $Comp
-L R R?
+L R R
 U 1 1 57CC7DA4
 P 4950 4800
-F 0 "R?" V 5030 4800 50  0000 C CNN
-F 1 "R" V 4950 4800 50  0000 C CNN
+F 0 "R" V 5030 4800 50  0000 C CNN
+F 1 "140" V 4950 4800 50  0000 C CNN
 F 2 "" V 4880 4800 50  0000 C CNN
 F 3 "" H 4950 4800 50  0000 C CNN
@@
 AC-live-f
 $Comp
-L R 100~ohm~NTC
+L R U?
 U 1 1 57CC96A4
 P 6800 4750
-F 0 "100 ohm NTC" V 6880 4750 50  0000 C CNN
-F 1 "R" V 6800 4750 50  0000 C CNN
+F 0 "U?" V 6880 4750 50  0000 C CNN
+F 1 "50 ohm NTC" V 6800 4750 50  0000 C CNN
 F 2 "" V 6730 4750 50  0000 C CNN
 F 3 "" H 6800 4750 50  0000 C CNN
@@
 $Comp
 L LM393 U?
-U 2 1 57CCA21B
+U 1 1 57CCA21B
 P 3850 6700
 F 0 "U?" H 4000 6850 50  0000 C CNN
@@
 F 2 "" H 3850 6700 50  0000 C CNN
 F 3 "" H 3850 6700 50  0000 C CNN
-	2    3850 6700
-	1    0    0    -1
-$EndComp
-$Comp
-L R MOV
+	1    3850 6700
+	1    0    0    -1
+$EndComp
+$Comp
+L R MOV?
 U 1 1 57CCAE9C
 P 2650 1050
-F 0 "MOV" V 2730 1050 50  0000 C CNN
-F 1 "R" V 2650 1050 50  0000 C CNN
+F 0 "MOV?" V 2730 1050 50  0000 C CNN
+F 1 "MOV" V 2650 1050 50  0000 C CNN
 F 2 "" V 2580 1050 50  0000 C CNN
 F 3 "" H 2650 1050 50  0000 C CNN
@@
 Connection ~ 3100 4900
 Connection ~ 1600 5100
-Wire Wire Line
-	1400 5100 1600 5100
 Wire Wire Line
 	1600 5100 3550 5100
@@
 $EndComp
 $Comp
-L R 0
+L R R
 U 1 1 57CE8283
 P 6300 2400
-F 0 "0 ohm" V 6380 2400 50  0000 C CNN
-F 1 "R" V 6300 2400 50  0000 C CNN
+F 0 "R" V 6380 2400 50  0000 C CNN
+F 1 "0" V 6300 2400 50  0000 C CNN
 F 2 "" V 6230 2400 50  0000 C CNN
 F 3 "" H 6300 2400 50  0000 C CNN
