File: inrush-limiter2/main.kicad_pcb (KiCad board)
At the start: 2 copper layers, 32 parts, among them K1 RELAY_2RT, P1 CONN_01X04, P2 CONN_01X02, Q1 2N3904, Q2 PN2222A, T1 TRANSFO, U1 LM393, U2 50 ohm NTC

Commit message: update
Parts:
- moved T1 7.41 mm to (168.9, 33.0), turned to 90 degrees
- moved R7 3.81 mm to (158.8, 59.7)
- moved P1 2.54 mm to (195.6, 61.0)
- moved R8 1.27 mm to (172.7, 59.7)
- moved F1 1.27 mm to (177.8, 81.3)
Routing:
- net AC-live-out: track 16.1 -> 59.8 mm
- net AC-neut: track 0.00 -> 23.4 mm
- net AC-live-f-low: track 11.7 -> 26.8 mm
- net Net-(F1-Pad2): track 0.43 -> 14.4 mm
Other:
- net class power: clearance 2 -> 1.75

Commit message: update
Parts:
- moved T1 10.8 mm to (176.5, 25.4)
- moved P2 6.84 mm to (149.9, 41.9)
Routing:
- net AC-live-f-low: track 26.8 -> 37.5 mm
- net AC-live-f: track 31.1 -> 27.0 mm
- net Net-(D2-Pad2): track 25.9 -> 27.1 mm
Changed lines of the file:
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@@
   (general
     (links 58)
-    (no_connects 4)
+    (no_connects 5)
     (area 110.105 17.444899 205.148001 96.28099)
     (thickness 1.6)
@@
   )
   (module Transformers_CHK:Trafo_CHK-EI30-2VA_Neutral (layer F.Cu)
-    (at 168.91 33.02 90)
+    (at 176.53 25.4 90)
     (descr "Trafo, Printtrafo, CHK, EI30, 2VA, neutral,")
     (tags "Trafo, Printtrafo, CHK, EI30, 2VA, neutral,")
@@
   )
   (module Wire_Pads:SolderWirePad_2x_1-2mmDrill (layer F.Cu)
-    (at 156.21 44.45 270)
+    (at 149.86 41.91 270)
     (fp_text reference P2 (at 0 -3.81 270) (layer F.SilkS)
       (effects (font (size 1 1) (thickness 0.15)))
@@
   (segment (start 123.19254 67.31052) (end 123.19 67.30798) (width 1) (layer B.Cu) (net 2) (status 30))
   (segment (start 146.04798 69.85) (end 146.04746 69.84948) (width 1) (layer B.Cu) (net 2) (status 30))
-  (segment (start 172.72 64.77) (end 176.53 67.31) (width 2.5) (layer B.Cu) (net 3) (status 10))
-  (segment (start 176.53 67.31) (end 175.26 66.04) (width 2.5) (layer B.Cu) (net 3))
-  (segment (start 170.18 66.04) (end 166.37 59.69) (width 2.5) (layer B.Cu) (net 3) (status 20))
+  (segment (start 177.8 70.27926) (end 177.8 69.85) (width 2.5) (layer B.Cu) (net 3) (status C00000))
+  (segment (start 177.8 69.85) (end 173.99 66.04) (width 2.5) (layer B.Cu) (net 3) (status 400000))
+  (segment (start 173.99 66.04) (end 170.18 66.04) (width 2.5) (layer B.Cu) (net 3) (status 800000))
+  (segment (start 166.37 59.69) (end 166.37 66.04) (width 2.5) (layer B.Cu) (net 3) (status 400000))
+  (segment (start 172.72 66.04) (end 172.72 64.77) (width 2.5) (layer B.Cu) (net 3) (status 800000))
+  (segment (start 172.72 66.04) (end 170.18 66.04) (width 2.5) (layer B.Cu) (net 3) (status 20))
   (segment (start 177.8 70.27926) (end 177.8 69.85) (width 2.5) (layer B.Cu) (net 3) (status 30))
-  (segment (start 177.8 69.85) (end 175.26 66.04) (width 2.5) (layer B.Cu) (net 3) (status 10))
-  (segment (start 175.26 66.04) (end 170.18 66.04) (width 2.5) (layer B.Cu) (net 3) (status 20))
-  (segment (start 177.8 70.27926) (end 177.8 69.85) (width 2.5) (layer B.Cu) (net 3) (status 30))
-  (segment (start 170.18 66.04) (end 163.83 66.04) (width 2.5) (layer B.Cu) (net 3) (status 30))
+  (segment (start 170.18 66.04) (end 166.37 66.04) (width 2.5) (layer B.Cu) (net 3) (status 30))
+  (segment (start 166.37 66.04) (end 163.83 66.04) (width 2.5) (layer B.Cu) (net 3) (status 30))
   (segment (start 177.8 70.27926) (end 178.22926 70.27926) (width 2.5) (layer B.Cu) (net 3) (status 30))
-  (segment (start 156.21 42.545) (end 156.21 46.355) (width 1) (layer B.Cu) (net 4))
   (segment (start 146.04746 59.68948) (end 147.32052 59.68948) (width 1) (layer B.Cu) (net 4))
-  (segment (start 156.21 50.8) (end 156.21 46.355) (width 1) (layer B.Cu) (net 4))
+  (segment (start 156.21 50.8) (end 149.86 43.815) (width 1) (layer B.Cu) (net 4) (status 20))
   (segment (start 147.32052 59.68948) (end 156.21 50.8) (width 1) (layer B.Cu) (net 4))
   (segment (start 142.24254 59.69052) (end 146.04642 59.69052) (width 1) (layer B.Cu) (net 4) (status 30))
@@
   (segment (start 171.45 71.12) (end 163.83 71.12) (width 2.5) (layer B.Cu) (net 5))
   (segment (start 182.88 82.55) (end 171.45 71.12) (width 2.5) (layer B.Cu) (net 5))
+  (segment (start 182.88 64.77) (end 180.34 62.23) (width 2.5) (layer B.Cu) (net 6) (status 400000))
+  (segment (start 180.34 62.23) (end 180.34 59.69) (width 2.5) (layer B.Cu) (net 6) (status 800000))
   (segment (start 189.611 77.47) (end 189.611 67.945) (width 2.5) (layer B.Cu) (net 6))
   (segment (start 189.611 67.945) (end 186.436 64.77) (width 2.5) (layer B.Cu) (net 6))
   (segment (start 186.436 64.77) (end 182.88 64.77) (width 2.5) (layer B.Cu) (net 6))
-  (segment (start 182.88 64.77) (end 181.61 63.5) (width 2.5) (layer B.Cu) (net 6))
-  (segment (start 181.61 63.5) (end 180.34 59.69) (width 2.5) (layer B.Cu) (net 6) (status 20))
   (segment (start 142.24 83.82) (end 142.24 90.17) (width 1) (layer B.Cu) (net 7) (status 30))
   (segment (start 134.62 93.98) (end 140.97 93.98) (width 1) (layer B.Cu) (net 7))
@@
   (segment (start 115.57 71.12) (end 114.3 72.39) (width 1) (layer B.Cu) (net 8))
   (segment (start 170.18 76.2) (end 163.83 76.2) (width 2.5) (layer B.Cu) (net 9) (status 30))
-  (segment (start 158.75 59.69) (end 179.07 44.45) (width 0.75) (layer B.Cu) (net 11) (status 10))
-  (segment (start 179.07 44.45) (end 178.90998 43.01998) (width 0.75) (layer B.Cu) (net 11) (status 30))
+  (segment (start 158.75 59.69) (end 186.69 36.83) (width 0.75) (layer B.Cu) (net 11) (status 20))
+  (segment (start 186.69 36.83) (end 186.52998 35.39998) (width 0.75) (layer B.Cu) (net 11) (status 30))
   (segment (start 147.32 83.82) (end 149.86 88.9) (width 1) (layer B.Cu) (net 12) (status 20))
   (segment (start 130.81 54.61) (end 130.81 57.15) (width 1) (layer B.Cu) (net 13) (status 10))

Commit message: add pin headers
Parts:
- P2: footprint Wire_Pads:SolderWirePad_2x_1-2mmDrill -> Pin_Headers:Pin_Header_Straight_1x02
- moved P2 37.5 mm to (134.6, 76.2)
Connections:
- P2 pad 1: Net-(D2-Pad2) -> GND
Routing:
- net AC-live-f-low: track 37.5 -> 1.44 mm
- net Net-(D2-Pad2): track 27.1 -> 5.08 mm
- net GND: track 242.2 -> 248.3 mm
- net +5V: track 84.7 -> 89.6 mm
Changed lines of the file:
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@@
     (links 58)
     (no_connects 5)
-    (area 110.105 17.444899 205.148001 96.28099)
+    (area 110.105 9.824899 205.148001 96.28099)
     (thickness 1.6)
     (drawings 0)
-    (tracks 157)
+    (tracks 165)
     (zones 0)
     (modules 32)
@@
     )
   )
-  (module Wire_Pads:SolderWirePad_2x_1-2mmDrill (layer F.Cu)
-    (at 149.86 41.91 270)
-    (fp_text reference P2 (at 0 -3.81 270) (layer F.SilkS)
-      (effects (font (size 1 1) (thickness 0.15)))
-    )
-    (fp_text value CONN_01X02 (at 0.635 3.81 270) (layer F.Fab)
-      (effects (font (size 1 1) (thickness 0.15)))
-    )
-    (pad 1 thru_hole circle (at -1.905 0 270) (size 2.99974 2.99974) (drill 1.19888) (layers *.Cu *.Mask F.SilkS)
-      (net 4 "Net-(D2-Pad2)"))
-    (pad 1 thru_hole circle (at 1.905 0 270) (size 2.99974 2.99974) (drill 1.19888) (layers *.Cu *.Mask F.SilkS)
-      (net 4 "Net-(D2-Pad2)"))
-  )
   (module test:fuck (layer F.Cu)
     (at 195.58 60.96 270)
@@
       (net 23 "Net-(F1-Pad2)"))
   )
+  (module Pin_Headers:Pin_Header_Straight_1x02 (layer F.Cu)
+    (at 134.62 76.2 270)
+    (descr "Through hole pin header")
+    (tags "pin header")
+    (fp_text reference P2 (at 0 -5.1 270) (layer F.SilkS)
+      (effects (font (size 1 1) (thickness 0.15)))
+    )
+    (fp_text value CONN_01X02 (at 0 -3.1 270) (layer F.Fab)
+      (effects (font (size 1 1) (thickness 0.15)))
+    )
+    (fp_line (start 1.27 1.27) (end 1.27 3.81) (layer F.SilkS) (width 0.15))
+    (fp_line (start 1.55 -1.55) (end 1.55 0) (layer F.SilkS) (width 0.15))
+    (fp_line (start -1.75 -1.75) (end -1.75 4.3) (layer F.CrtYd) (width 0.05))
+    (fp_line (start 1.75 -1.75) (end 1.75 4.3) (layer F.CrtYd) (width 0.05))
+    (fp_line (start -1.75 -1.75) (end 1.75 -1.75) (layer F.CrtYd) (width 0.05))
+    (fp_line (start -1.75 4.3) (end 1.75 4.3) (layer F.CrtYd) (width 0.05))
+    (fp_line (start 1.27 1.27) (end -1.27 1.27) (layer F.SilkS) (width 0.15))
+    (fp_line (start -1.55 0) (end -1.55 -1.55) (layer F.SilkS) (width 0.15))
+    (fp_line (start -1.55 -1.55) (end 1.55 -1.55) (layer F.SilkS) (width 0.15))
+    (fp_line (start -1.27 1.27) (end -1.27 3.81) (layer F.SilkS) (width 0.15))
+    (fp_line (start -1.27 3.81) (end 1.27 3.81) (layer F.SilkS) (width 0.15))
+    (pad 1 thru_hole rect (at 0 0 270) (size 2.032 2.032) (drill 1.016) (layers *.Cu *.Mask F.SilkS)
+      (net 2 GND))
+    (pad 2 thru_hole oval (at 0 2.54 270) (size 2.032 2.032) (drill 1.016) (layers *.Cu *.Mask F.SilkS)
+      (net 22 +5V))
+    (model Pin_Headers.3dshapes/Pin_Header_Straight_1x02.wrl
+      (at (xyz 0 -0.05 0))
+      (scale (xyz 1 1 1))
+      (rotate (xyz 0 0 90))
+    )
+  )
   (segment (start 133.35 54.61) (end 134.62 55.88) (width 1) (layer B.Cu) (net 1) (status 10))
   (segment (start 134.62 55.88) (end 134.62 59.69) (width 1) (layer B.Cu) (net 1) (status 20))
@@
   (segment (start 142.24202 69.85) (end 142.24254 69.85052) (width 1) (layer B.Cu) (net 1) (status 30))
   (segment (start 138.43 69.84798) (end 138.43254 69.85052) (width 1) (layer B.Cu) (net 1) (status 30))
+  (segment (start 134.625 72.385) (end 132.085 72.385) (width 1) (layer B.Cu) (net 2))
+  (segment (start 130.82 71.12) (end 130.82 67.31) (width 1) (layer B.Cu) (net 2) (status 800000))
+  (segment (start 132.085 72.385) (end 130.82 71.12) (width 1) (layer B.Cu) (net 2))
+  (segment (start 135.895 72.385) (end 134.625 72.385) (width 1) (layer B.Cu) (net 2))
+  (segment (start 134.625 72.385) (end 134.62 76.2) (width 1) (layer B.Cu) (net 2) (status 20))
   (segment (start 120.65 85.09) (end 120.65 87.63) (width 1) (layer B.Cu) (net 2) (status 10))
   (segment (start 120.65 87.63) (end 125.73 92.71) (width 1) (layer B.Cu) (net 2) (status 20))
@@
   (segment (start 146.04746 69.84948) (end 146.04746 69.85254) (width 1) (layer B.Cu) (net 2) (status 30))
   (segment (start 146.04746 69.85254) (end 143.51 72.39) (width 1) (layer B.Cu) (net 2) (status 10))
-  (segment (start 135.9 72.39) (end 130.82 67.31) (width 1) (layer B.Cu) (net 2) (status 20))
+  (segment (start 135.9 72.39) (end 135.895 72.385) (width 1) (layer B.Cu) (net 2) (status 20))
   (segment (start 143.51 72.39) (end 135.9 72.39) (width 1) (layer B.Cu) (net 2))
   (segment (start 130.82 67.31) (end 123.19 67.31) (width 1) (layer B.Cu) (net 2) (status 30))
@@
   (segment (start 123.19254 67.31052) (end 123.19 67.30798) (width 1) (layer B.Cu) (net 2) (status 30))
   (segment (start 146.04798 69.85) (end 146.04746 69.84948) (width 1) (layer B.Cu) (net 2) (status 30))
-  (segment (start 177.8 70.27926) (end 177.8 69.85) (width 2.5) (layer B.Cu) (net 3) (status C00000))
-  (segment (start 177.8 69.85) (end 173.99 66.04) (width 2.5) (layer B.Cu) (net 3) (status 400000))
-  (segment (start 173.99 66.04) (end 170.18 66.04) (width 2.5) (layer B.Cu) (net 3) (status 800000))
-  (segment (start 166.37 59.69) (end 166.37 66.04) (width 2.5) (layer B.Cu) (net 3) (status 400000))
-  (segment (start 172.72 66.04) (end 172.72 64.77) (width 2.5) (layer B.Cu) (net 3) (status 800000))
+  (segment (start 177.8 70.27926) (end 177.8 69.85) (width 2.5) (layer B.Cu) (net 3))
+  (segment (start 177.8 69.85) (end 173.99 66.04) (width 2.5) (layer B.Cu) (net 3))
+  (segment (start 173.99 66.04) (end 170.18 66.04) (width 2.5) (layer B.Cu) (net 3))
+  (segment (start 166.37 59.69) (end 166.37 66.04) (width 2.5) (layer B.Cu) (net 3))
+  (segment (start 172.72 66.04) (end 172.72 64.77) (width 2.5) (layer B.Cu) (net 3))
   (segment (start 172.72 66.04) (end 170.18 66.04) (width 2.5) (layer B.Cu) (net 3) (status 20))
   (segment (start 177.8 70.27926) (end 177.8 69.85) (width 2.5) (layer B.Cu) (net 3) (status 30))
@@
   (segment (start 177.8 70.27926) (end 178.22926 70.27926) (width 2.5) (layer B.Cu) (net 3) (status 30))
   (segment (start 146.04746 59.68948) (end 147.32052 59.68948) (width 1) (layer B.Cu) (net 4))
-  (segment (start 156.21 50.8) (end 149.86 43.815) (width 1) (layer B.Cu) (net 4) (status 20))
-  (segment (start 147.32052 59.68948) (end 156.21 50.8) (width 1) (layer B.Cu) (net 4))
   (segment (start 142.24254 59.69052) (end 146.04642 59.69052) (width 1) (layer B.Cu) (net 4) (status 30))
   (segment (start 146.04642 59.69052) (end 146.04746 59.68948) (width 1) (layer B.Cu) (net 4) (status 30))
@@
   (segment (start 171.45 71.12) (end 163.83 71.12) (width 2.5) (layer B.Cu) (net 5))
   (segment (start 182.88 82.55) (end 171.45 71.12) (width 2.5) (layer B.Cu) (net 5))
-  (segment (start 182.88 64.77) (end 180.34 62.23) (width 2.5) (layer B.Cu) (net 6) (status 400000))
-  (segment (start 180.34 62.23) (end 180.34 59.69) (width 2.5) (layer B.Cu) (net 6) (status 800000))
+  (segment (start 182.88 64.77) (end 180.34 62.23) (width 2.5) (layer B.Cu) (net 6))
+  (segment (start 180.34 62.23) (end 180.34 59.69) (width 2.5) (layer B.Cu) (net 6))
   (segment (start 189.611 77.47) (end 189.611 67.945) (width 2.5) (layer B.Cu) (net 6))
   (segment (start 189.611 67.945) (end 186.436 64.77) (width 2.5) (layer B.Cu) (net 6))
@@
   (segment (start 115.57 71.12) (end 114.3 72.39) (width 1) (layer B.Cu) (net 8))
   (segment (start 170.18 76.2) (end 163.83 76.2) (width 2.5) (layer B.Cu) (net 9) (status 30))
-  (segment (start 158.75 59.69) (end 186.69 36.83) (width 0.75) (layer B.Cu) (net 11) (status 20))
   (segment (start 186.69 36.83) (end 186.52998 35.39998) (width 0.75) (layer B.Cu) (net 11) (status 30))
   (segment (start 147.32 83.82) (end 149.86 88.9) (width 1) (layer B.Cu) (net 12) (status 20))
@@
   (segment (start 123.19 86.36) (end 125.73 88.9) (width 1) (layer B.Cu) (net 21))
   (segment (start 121.92 76.2) (end 120.65 76.2) (width 1) (layer B.Cu) (net 21) (status 20))
+  (segment (start 132.08 76.2) (end 132.08 78.74) (width 1) (layer B.Cu) (net 22) (status 400000))
+  (segment (start 129.54 78.74) (end 130.81 78.74) (width 1) (layer B.Cu) (net 22))
+  (segment (start 125.73 73.66) (end 125.73 76.2) (width 1) (layer B.Cu) (net 22))
+  (segment (start 125.73 76.2) (end 128.27 78.74) (width 1) (layer B.Cu) (net 22))
+  (segment (start 128.27 78.74) (end 130.81 78.74) (width 1) (layer B.Cu) (net 22))
+  (segment (start 130.81 78.74) (end 132.08 78.74) (width 1) (layer B.Cu) (net 22))
+  (segment (start 132.08 78.74) (end 137.16 78.74) (width 1) (layer B.Cu) (net 22))
   (segment (start 116.84 63.5) (end 116.84 67.31) (width 1) (layer B.Cu) (net 22) (status 10))
   (segment (start 116.84 59.69) (end 114.3 59.69) (width 1) (layer B.Cu) (net 22) (status 10))
@@
   (segment (start 114.3 59.69) (end 114.3 60.96) (width 1) (layer B.Cu) (net 22))
   (segment (start 115.57 55.88) (end 114.3 57.15) (width 1) (layer B.Cu) (net 22))
-  (segment (start 125.73 73.66) (end 125.73 76.2) (width 1) (layer B.Cu) (net 22) (status 10))
   (segment (start 116.84 67.31) (end 125.73 76.2) (width 1) (layer B.Cu) (net 22))
-  (segment (start 125.73 76.2) (end 137.16 76.2) (width 1) (layer B.Cu) (net 22))
   (segment (start 147.32 76.2) (end 149.86 76.2) (width 1) (layer B.Cu) (net 22) (status 10))
   (segment (start 149.86 76.2) (end 163.83 90.17) (width 1) (layer B.Cu) (net 22) (status 20))
   (segment (start 163.83 90.17) (end 163.83 91.44) (width 1) (layer B.Cu) (net 22) (status 30))
-  (segment (start 137.16 76.2) (end 137.16 83.82) (width 1) (layer B.Cu) (net 22) (status 20))
+  (segment (start 137.16 76.2) (end 137.16 78.74) (width 1) (layer B.Cu) (net 22) (status 20))
+  (segment (start 137.16 78.74) (end 137.16 83.82) (width 1) (layer B.Cu) (net 22) (status 20))
   (segment (start 142.24 76.2) (end 137.16 76.2) (width 1) (layer B.Cu) (net 22) (status 10))
   (segment (start 147.32 76.2) (end 142.24 76.2) (width 1) (layer B.Cu) (net 22) (status 30))
